File: AudioSystemEQPanel/AudioSystemEQPanel.kicad_sch (KiCad schematic)
At the start: 46 parts, among them J1 AudioJack3, U1 OPA2134, U2 OPA2134, U3 OPA2134, U4 OPA2134

Commit message: fixed symbol lab problem, added symbols to all ics
Parts:
- U1, U2, U3, U4: footprint (none) -> AudioSystemFootprintLibrary:OPA2134UA
Changed lines of the file:
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@@
 			)
 		)
-		(property "Footprint" ""
+		(property "Footprint" "AudioSystemFootprintLibrary:OPA2134UA"
 			(at 82.55 148.59 0)
 			(effects
@@
 			)
 		)
-		(property "Footprint" ""
+		(property "Footprint" "AudioSystemFootprintLibrary:OPA2134UA"
 			(at 290.83 100.33 0)
 			(effects
@@
 			)
 		)
-		(property "Footprint" ""
+		(property "Footprint" "AudioSystemFootprintLibrary:OPA2134UA"
 			(at 144.78 254 0)
 			(effects
@@
 			)
 		)
-		(property "Footprint" ""
+		(property "Footprint" "AudioSystemFootprintLibrary:OPA2134UA"
 			(at 82.55 100.33 0)
 			(effects
@@
 			)
 		)
-		(property "Footprint" ""
+		(property "Footprint" "AudioSystemFootprintLibrary:OPA2134UA"
 			(at 170.18 100.33 0)
 			(effects
@@
 			)
 		)
-		(property "Footprint" ""
+		(property "Footprint" "AudioSystemFootprintLibrary:OPA2134UA"
 			(at 100.33 254 0)
 			(effects
@@
 			)
 		)
-		(property "Footprint" ""
+		(property "Footprint" "AudioSystemFootprintLibrary:OPA2134UA"
 			(at 194.31 255.27 0)
 			(effects
@@
 			)
 		)
-		(property "Footprint" ""
+		(property "Footprint" "AudioSystemFootprintLibrary:OPA2134UA"
 			(at 290.83 148.59 0)
 			(effects
@@
 			)
 		)
-		(property "Footprint" ""
+		(property "Footprint" "AudioSystemFootprintLibrary:OPA2134UA"
 			(at 170.18 148.59 0)
 			(effects
@@
 			)
 		)
-		(property "Footprint" ""
+		(property "Footprint" "AudioSystemFootprintLibrary:OPA2134UA"
 			(at 242.57 100.33 0)
 			(effects
@@
 			)
 		)
-		(property "Footprint" ""
+		(property "Footprint" "AudioSystemFootprintLibrary:OPA2134UA"
 			(at 242.57 148.59 0)
 			(effects
@@
 			)
 		)
-		(property "Footprint" ""
+		(property "Footprint" "AudioSystemFootprintLibrary:OPA2134UA"
 			(at 50.8 254 0)
 			(effects

Commit message: changed all panels input and output audio interfaces, added noisecancellation panel
Parts:
- added J2: AudioJack3, symbol Connector_Audio:AudioJack3
Connections:
- net GND: now also J2.S
- net at R21.2, U4.1: now also J2.T
- net at R24.2, U4.7: now also J2.R
Changed lines of the file:
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@@
 	)
 	(junction
+		(at 300.99 100.33)
+		(diameter 0)
+		(color 0 0 0 0)
+	)
+	(junction
 		(at 283.21 139.7)
 		(diameter 0)
@@
 	)
 	(junction
+		(at 300.99 148.59)
+		(diameter 0)
+		(color 0 0 0 0)
+	)
+	(junction
 		(at 234.95 109.22)
 		(diameter 0)
@@
 	(wire
 		(pts
+			(xy 300.99 100.33) (xy 320.04 100.33)
+		)
+		(stroke
+			(width 0)
+			(type default)
+		)
+	)
+	(wire
+		(pts
 			(xy 176.53 109.22) (xy 180.34 109.22)
 		)
@@
 	(wire
 		(pts
+			(xy 320.04 123.19) (xy 349.25 123.19)
+		)
+		(stroke
+			(width 0)
+			(type default)
+		)
+	)
+	(wire
+		(pts
 			(xy 57.15 151.13) (xy 60.96 151.13)
 		)
@@
 	(wire
 		(pts
+			(xy 320.04 100.33) (xy 320.04 123.19)
+		)
+		(stroke
+			(width 0)
+			(type default)
+		)
+	)
+	(wire
+		(pts
 			(xy 271.78 144.78) (xy 271.78 139.7)
 		)
@@
 	(wire
 		(pts
+			(xy 320.04 125.73) (xy 349.25 125.73)
+		)
+		(stroke
+			(width 0)
+			(type default)
+		)
+	)
+	(wire
+		(pts
 			(xy 53.34 200.66) (xy 53.34 210.82)
 		)
@@
 	(wire
 		(pts
+			(xy 320.04 148.59) (xy 320.04 125.73)
+		)
+		(stroke
+			(width 0)
+			(type default)
+		)
+	)
+	(wire
+		(pts
 			(xy 92.71 180.34) (xy 180.34 180.34)
 		)
@@
 	(wire
 		(pts
+			(xy 349.25 128.27) (xy 349.25 138.43)
+		)
+		(stroke
+			(width 0)
+			(type default)
+		)
+	)
+	(wire
+		(pts
 			(xy 92.71 171.45) (xy 92.71 180.34)
 		)
@@
 	(wire
 		(pts
+			(xy 300.99 148.59) (xy 320.04 148.59)
+		)
+		(stroke
+			(width 0)
+			(type default)
+		)
+	)
+	(wire
+		(pts
 			(xy 48.26 200.66) (xy 53.34 200.66)
 		)
@@
 	)
 	(symbol
+		(lib_id "power:GND")
+		(at 349.25 138.43 0)
+		(unit 1)
+		(exclude_from_sim no)
+		(in_bom yes)
+		(on_board yes)
+		(dnp no)
+		(fields_autoplaced yes)
+		(property "Reference" "#PWR018"
+			(at 349.25 144.78 0)
+			(effects
+				(font
+					(size 1.27 1.27)
+				)
+				(hide yes)
+			)
+		)
+		(property "Value" "GND"
+			(at 349.25 143.51 0)
+			(effects
+				(font
+					(size 1.27 1.27)
+				)
+			)
+		)
+		(property "Footprint" ""
+			(at 349.25 138.43 0)
+			(effects
+				(font
+					(size 1.27 1.27)
+				)
+				(hide yes)
+			)
+		)
+		(property "Datasheet" ""
+			(at 349.25 138.43 0)
+			(effects
+				(font
+					(size 1.27 1.27)
+				)
+				(hide yes)
+			)
+		)
+		(property "Description" "Power symbol creates a global label with name \"GND\" , ground"
+			(at 349.25 138.43 0)
+			(effects
+				(font
+					(size 1.27 1.27)
+				)
+				(hide yes)
+			)
+		)
+		(pin "1"
+		)
+		(instances
+			(project "AudioSystemEQPanel"
+				(path "/d171f5e5-58fa-445c-b596-876d1e770727"
+					(reference "#PWR018")
+					(unit 1)
+				)
+			)
+		)
+	)
+	(symbol
 		(lib_id "Device:R")
 		(at 180.34 167.64 180)
@@
 					(unit 1)
 				)
+			)
+		)
+	)
+	(symbol
+		(lib_id "Connector_Audio:AudioJack3")
+		(at 354.33 125.73 180)
+		(unit 1)
+		(exclude_from_sim no)
+		(in_bom yes)
+		(on_board yes)
+		(dnp no)
+		(fields_autoplaced yes)
+		(property "Reference" "J2"
+			(at 361.95 123.8249 0)
+			(effects
+				(font
+					(size 1.27 1.27)
+				)
+				(justify right)
+			)
+		)
+		(property "Value" "AudioJack3"
+			(at 361.95 126.3649 0)
+			(effects
+				(font
+					(size 1.27 1.27)
+				)
+				(justify right)
+			)
+		)
+		(property "Footprint" ""
+			(at 354.33 125.73 0)
+			(effects
+				(font
+					(size 1.27 1.27)
+				)
+				(hide yes)
+			)
+		)
+		(property "Datasheet" "~"
+			(at 354.33 125.73 0)
+			(effects
+				(font
+					(size 1.27 1.27)
+				)
+				(hide yes)
+			)
+		)
+		(property "Description" "Audio Jack, 3 Poles (Stereo / TRS)"
+			(at 354.33 125.73 0)
+			(effects
+				(font
+					(size 1.27 1.27)
+				)
+				(hide yes)
+			)
+		)
+		(pin "T"
+		)
+		(pin "R"
+		)
+		(pin "S"
+		)
+		(instances
+			(project ""
+				(path "/d171f5e5-58fa-445c-b596-876d1e770727"
+					(reference "J2")
+					(unit 1)
+				)
