File: Schematics/AudioSystemFull/AudioSystemFull.kicad_sch (KiCad schematic)
At the start: 88 parts, among them IC1 TDA1558Q, J1 AudioJack3, U1 OPA2134, U10 MAX660ESA, U11 LM7805_TO220, U12 MAX660ESA, U2 DEVKIT_V1_ESP32-WROOM-32, U3 PCM5102A, U4 OPA2134, U5 OPA2134, U6 OPA2134, U7 OPA2134, U8 OPA2134, U9 LM7805_TO220

Commit message: a2dp sink, avrcp data displaying and animating on lcd done
Parts:
- added C33, C34: 10u, symbol Device:C_Polarized_Small_US
- added U13: LM1085-3.3, symbol Regulator_Linear:LM1085-3.3
Connections:
- net +3.3VA is gone; now on net +3.3VMain: C10.2, C11.1, C12.1, C8.2, U3.1 (CPVDD), U3.17 (XSMT), U3.8 (AVDD)
- net +5V is gone; now on net +5VMain: R1.2, R3.2
- net GND: now also C10.1, C11.2, C12.2, C8.1, C9.2, U2.14 (GND1), U3.3 (CPGND), U3.9 (AGND)
- net GNDA: no longer C10.1, C11.2, C12.2, C8.1, C9.2, U3.3 (CPGND), U3.9 (AGND)
- net GNDPWR: now also C33.2, C34.2, U13.1 (GND)
- net +12V: now reaches C29.1, U9.1 (VI)
- net +12V: now also C31.1, U11.1 (VI), C33.1, U13.3 (VI)
- net -5VMain: now reaches U7.4 (V-)
- net -5VMain: now also U1.4 (V-), U10.5 (OUT), U4.4 (V-), U5.4 (V-), U6.4 (V-), U8.4 (V-)
- net +5VMain: now reaches U7.8 (V+)
- net +5VMain: now also C30.1, U1.8 (V+), U10.1 (FC), U10.8 (V+), U2.19 (EXT_5V), U4.8 (V+), U5.8 (V+), U6.8 (V+), U8.8 (V+), U9.3 (VO)
- net +5VMic: now reaches C32.1, U11.3 (VO), U12.1 (FC), U12.8 (V+)
- net -5VMic: now reaches U12.5 (OUT)
- net +3.3V renamed +3.3VMain
- net +3.3VMain: now also C34.1, U13.2 (VO)
- net +AAOutL renamed +AAL
- net +AAOutR renamed +AAR
- net -AAOutL renamed -AAL
- net -AAOutR renamed -AAR
- net FAOutL renamed FAL
- net FAOutR renamed FAR
- net L_HIGH renamed RAHighL
- net L_LOW renamed RALowL
- net L_MID renamed RAMidL
- net R_HIGH renamed RAHighR
- net R_LOW renamed RALowR
- net R_MID renamed RAMidR
Other:
- note added: "RALowL - Raw Audio Low frequency Left channel RAMidL - Raw Audio Mid frequency Left channel RAHighL - Raw Audio High frequency Left channel RALowR - Raw Audio Low frequency Right channel RAMidR - Raw Audio Mid frequency Right channel RAHighR - Raw Audio High frequency Right channel FAL - Filtered Audio Left channel FAR - Filtered Audio Right channel +AAL - Amplified Audio Left channel Positive -A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"
- moved on the sheet: C15, C16, C17, C18, C19, C20, C21, C22, C27, C28, C31, C32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

Commit message: progress check
Parts:
- removed J1: AudioJack3, symbol Connector_Audio:AudioJack3
- removed R2, R4: 500k, symbol Device:R
- removed U1: OPA2134, AudioSystemFootprintLibrary:OPA2134UA, symbol Amplifier_Operational:OPA2134
- added J1: SJ1-3515-SMT-TR-BE, AudioSystemFootprintLibrary:SJ1-3515-SMT-TR-BE, symbol AudioSystemSymbolLibrary:SJ1-3515-SMT-TR-BE
- C1, C2: value 1u -> 2.2u
- R1, R3: value 2M -> 4.7k
- U10, U12: footprint MAX660ESA_:SOIC127P600X175-8N -> AudioSystemFootprintLibrary:MAX660ESA
- U13: footprint (none) -> AudioSystemFootprintLibrary:LM1085IT-3.3
Connections:
- net GNDPWR is gone; now on net GND: C25.1, C26.2, C29.2, C30.2, C31.2, C32.2, C33.2, C34.2, IC1.11 (GND2), IC1.7 (GND1), U10.3 (GND), U11.2 (GND), U12.3 (GND), U13.1 (GND), U9.2 (GND)
- net GNDS is gone; now on net GND: IC1.3 (GNDSIG)
- net +12V: no longer C33.1, U13.3 (VI)
- net +5VMain: now also C33.1, U13.3 (VI)
- net GND: now also R1.1, R3.1, U2.5 (IO34), U2.6 (IO35), J1.1, J1.10, J1.11
- net at C2.1: now also J1.3
- net at C1.1: now also J1.2
- net at R10.1: now also C2.2
- net at R8.1: now also C1.2
Other:
- moved on the sheet: C1, C2, C23, C24, C25, C26, IC1, R11, R12, R13, R14, R17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

Commit message: power supply schematic possibly done
Parts:
- removed C20: 22n, symbol Device:C_Small
- removed C27, C28, C33, C34: 10u, symbol Device:C_Polarized_Small_US
- removed R10, R21, R22, R37, R38, R7, R8, R9: 1k, symbol Device:R
- removed R15, R16, R25, R26: 27k, symbol Device:R
- removed R19, R20: 2k, symbol Device:R
- removed R23, R24, R31, R32: 3.6k, symbol Device:R
- removed R27, R28: 68k, symbol Device:R
- removed R29, R30: 510, symbol Device:R
- removed R33, R34: 2.6k, symbol Device:R
- removed R35, R36: 750, symbol Device:R
- removed RV1, RV2, RV3: 20k, symbol Device:R_Potentiometer_Dual
- removed RV4: 10k, symbol Device:R_Potentiometer_Dual
- removed U10, U12: MAX660ESA, AudioSystemFootprintLibrary:MAX660ESA, symbol AudioSystemSymbolLibrary:MAX660ESA
- removed U11, U9: LM7805_TO220, Package_TO_SOT_THT:TO-220-3_Vertical, symbol Regulator_Linear:LM7805_TO220
- removed U13: LM1085-3.3, AudioSystemFootprintLibrary:LM1085IT-3.3, symbol Regulator_Linear:LM1085-3.3
- removed U5, U6, U7, U8: OPA2134, AudioSystemFootprintLibrary:OPA2134UA, symbol Amplifier_Operational:OPA2134
- added C20: 10u, symbol Device:C_Polarized_Small_US
- added C27: 1u, symbol Device:C_Small
- added C28, C37: 1000u, symbol Device:C_Small
- added C33, C39, C47: 0.1u, symbol Device:C_Small
- added C34, C35, C36, C40, C41, C42: 10u, symbol Device:C_Small
- added C38, C46: 2.2u, symbol Device:C_Small
- added C43, C50, C51, C52, C53, C54, C55, C56, C57, C58, C59, C60: 22n, symbol Device:C_Small
- added C44, C45, C61, C62, C63, C64, C65, C66, C67, C68, C69, C70, C71, C72, C73, C74, C75, C76: 100n, symbol Device:C_Small
- added C48, C49: 22u, symbol Device:C_Small
- added J2: DISPLAY, symbol Connector:Conn_01x04_Pin
- added J3: ISO_Conn_Unit_B, symbol Connector:Conn_01x08_Pin
- added J4: ISO_Conn_Unit_A, symbol Connector:Conn_01x08_Pin
- added L1, L3, L6: 1u, symbol Device:L
- added L2: 3.3u, symbol Device:L
- added L4: 4.7u, symbol Device:L
- added L7: 10u, symbol Device:L
- added R10, R15, R45: 100k, symbol Device:R_Small
- added R16, R20, R21, R23, R29, R30, R31, R33, R49, R50, R51, R53: 5k, symbol Device:R_Small
- added R19: 160, symbol Device:R_Small
- added R2: 240, symbol Device:R_Small
- added R22, R24, R25, R26, R27, R28, R32, R34, R52, R54: 500, symbol Device:R_Small
- added R35, R37, R38, R42, R46: 12k, symbol Device:R_Small
- added R36, R43: 56k, symbol Device:R_Small
- added R39, R47: 2k, symbol Device:R_Small
- added R4: 11k, symbol Device:R_Small
- added R40, R44: 470, symbol Device:R
- added R41, R48, R59, R60, R61, R62, R63, R64, R65, R66: 1k, symbol Device:R_Small
- added R55, R56, R57, R58: 7.5k, symbol Device:R_Small
- added R7: 2.7k, symbol Device:R_Small
- added R8, R9: 10k, symbol Device:R_Small
- added RV1, RV2, RV3: 10k, symbol Device:R_Potentiometer_Dual_Separate
- added U1: LP3856ES-5.0, AudioSystemFootprintLibrary:LP3856ES-5.0, symbol AudioSystemSymbolLibrary:LP3856ES-5.0
- added U10: LT3015EQ-5PBF, AudioSystemFootprintLibrary:LT3015EQ-5PBF, symbol AudioSystemSymbolLibrary:LT3015EQ-5PBF
- added U11, U12, U13, U14, U15, U16, U17: OPA2134, symbol Amplifier_Operational:OPA2134
- added U5, U8: LP5907MFX-3.3, Package_TO_SOT_SMD:SOT-23-5, symbol Regulator_Linear:LP5907MFX-3.3
- added U6: LMR51420XFDDCR, AudioSystemFootprintLibrary:LMR51420XFDDCR, symbol AudioSystemSymbolLibrary:LMR51420XFDDCR
- added U7: LMR51420YFDDCR, AudioSystemFootprintLibrary:LMR51420YFDDCR, symbol AudioSystemSymbolLibrary:LMR51420YFDDCR
- added U9: LMR51430YFDDCR, AudioSystemFootprintLibrary:LMR51430YFDDCR, symbol AudioSystemSymbolLibrary:LMR51430YFDDCR
- C15, C16: value 22n -> 100n
- C17: value 22n -> 10n
- C18, C19, C22: value 22n -> 1u
- C21: value 22n -> 10u
- C29: value 0.33u -> 10n
- C30: value 0.1u -> 100n
- C31: value 0.33u -> 100n
- C32: value 0.1u -> 2.2u
Connections:
- net +5VMic is gone; now on an unnamed net: C32.1
- net Vcc is gone; now on net +12VPerm: C25.2, C26.1, IC1.13 (VCC1), IC1.5 (VCC)
- net FAL: now also R62.1, U17.1
- net FAR: now also R66.1, U17.7
- net GND: now also C22.2, C27.2, C44.2, C45.2, C46.2, C48.2, C49.2, J2.1 (Pin_1), J4.8 (Pin_8), R7.2, U6.1 (GND), U8.2 (GND); no longer C10.1, C11.2, C12.2, C15.2, C16.2, C19.2, C29.2, C30.2, C31.2, C32.2, C8.1, C9.2, IC1.11 (GND2), IC1.3 (GNDSIG), IC1.7 (GND1), J1.10, J1.11, R1.1, R11.1, R12.1, R13.1, R14.1, R17.1, R18.1, R3.1, U2.5 (IO34), U2.6 (IO35), U3.3 (CPGND), U3.9 (AGND), U4.1, U4.2 (-), U4.6 (-), U4.7
- net GNDA: now also C10.1, C11.2, C12.2, C15.2, C16.2, C17.2, C18.2, C19.2, C21.2, C29.2, C30.2, C31.2, C32.2, C8.1, C9.2, IC1.11 (GND2), IC1.3 (GNDSIG), IC1.7 (GND1), R11.1, R12.1, R13.1, R14.1, R17.1, R18.1, U3.3 (CPGND), U3.9 (AGND), U4.1, U4.2 (-), U4.6 (-), U4.7, C20.2, C28.2, C34.1, C35.1, C36.2, C37.2, C38.2, C40.2, C41.2, C42.2, C50.1, C51.1, C53.1, C55.1, C61.2, C62.2, C63.2, C64.2, C65.2, C66.2, C67.2, C68.2, C69.2, C70.2, C71.2, C72.2, C73.2, C74.2, C75.2, C76.2, L4.2, R19.1, R2.2, R21.1, R23.1, R31.1, R33.1, R37.2, R41.2, R42.2, R48.2, R51.1, R53.1, R55.2, R57.2, RV1.3, RV1.6, RV2.3, RV2.6, RV3.3, RV3.6, U1.3 (GND), U10.2 (GND), U17.3 (+), U17.6 (-), U5.2 (GND), U9.1 (GND)
- net RAHighL: now also R49.2; no longer C21.1
- net RAHighR: now also R50.2; no longer C22.1
- net RALowL: now also R16.2
- net RALowR: now also R20.2
- net RAMidL: now also R30.2; no longer C17.1
- net RAMidR: now also R29.2; no longer C18.1
- net +12VPerm: now reaches C15.1
- net +12VPerm: now also C17.1, C29.1, C30.1, C28.1, C37.1, C44.1, J4.4 (Pin_4), L1.1, L3.1, L6.1, U7.5 (EN)
- net +3.3VAnalog: now reaches C19.1
- net +3.3VAnalog: now also C10.2, C11.1, C12.1, C8.2, U3.1 (CPVDD), U3.8 (AVDD), U5.5 (OUT)
- net at C14.1, R6.2: now also U4.5 (+), R40.2
- net at C16.1: now also C38.1, L3.2, U9.3 (VIN), U9.5 (EN)
- net at C2.2: now also R40.1
- net at U4.3 (+): now also C13.1, R5.2, R44.2
- net at C1.2: now also R44.1
- net I2C_SDA: now reaches U2.27 (IO16)
- net I2C_SDA: now also J2.3 (Pin_3)
- net I2C_SCL: now reaches U2.28 (IO17)
- net I2C_SCL: now also J2.4 (Pin_4)
- net +12V: no longer names the net of C31.1
- net +12V: now also C34.2, C35.2, C36.1, L1.2, R10.2, U10.1 (*SHDN), U10.3 (IN), U10.6 (EPAD), U7.1 (GND), U7.3 (VIN); no longer C29.1
- removed net +3.3VMain: C10.2, C11.1, C12.1, C4.1, C6.2, C8.2, U3.1 (CPVDD), U3.17 (XSMT), U3.20 (DVDD), U3.8 (AVDD)
- net +5VMain renamed +5VDigital
- net +5VDigital: now also C22.1, C48.1, C49.1, J2.2 (Pin_2), L7.2, R15.1, U8.1 (IN), U8.3 (EN); no longer C30.1, U4.8 (V+)
- net +AAL renamed LeftFront+
- net LeftFront+: now also J3.5 (Pin_5)
- net +AAR renamed RightFront+
- net RightFront+: now also J3.3 (Pin_3)
- net -5VMain renamed -5VAnalog
- net -5VAnalog: now also C42.1, C62.1, C64.1, C66.1, C68.1, C70.1, C72.1, C74.1, C76.1, U10.4 (SENSE/ADJ), U10.5 (OUT), U11.4 (V-), U12.4 (V-), U13.4 (V-), U14.4 (V-), U15.4 (V-), U16.4 (V-), U17.4 (V-)
- net -AAL renamed LeftFront-
- net LeftFront-: now also J3.6 (Pin_6)
- net -AAR renamed RightFront-
- net RightFront-: now also J3.4 (Pin_4)
- new net: C45.1, C46.1, L6.2, U6.3 (VIN), U6.5 (EN)
- new net: C56.1, R42.1, U14.5 (+)
- new net: R47.2, R48.1, U14.6 (-)
- new net: R63.1, R64.1, R65.1, R66.2, U17.5 (+)
- new net: R10.1, R9.2, U7.4 (FB)
- new net: C55.2, C56.2, R38.1, R43.2
- new net: C52.1, R27.1, R28.2
- new net: R16.1, RV1.1
- new net: C43.1, R25.1, R26.2
- new net: R24.1, R25.2, U11.7
- new net: R49.1, RV3.1
- new net: RV3.2, U15.3 (+)
- new net: C53.2, C54.2, R35.1, R36.2
- new net: R32.1, R35.2, U13.1
- new net: R31.2, R32.2, U13.2 (-)
- new net: RV1.5, U11.5 (+)
- new net: R23.2, R24.2, U11.6 (-)
- new net: C18.1, C20.1, C40.1, C41.1, L2.2, R45.1, R8.1, U1.2 (IN), U5.1 (IN), U5.3 (EN)
- new net: C60.1, R57.1, U16.5 (+)
- new net: C59.1, C60.2, R58.1
- new net: R19.2, R9.1
- new net: RV2.2, U13.3 (+)
- new net: C58.1, R55.1, U16.3 (+)
- new net: R59.1, R60.1, R61.1, R62.2, U17.2 (-)
- new net: R30.1, RV2.1
- new net: RV1.2, U11.3 (+)
- new net: C57.1, C58.2, R56.1
- new net: C47.2, L7.1, U6.2 (SW)
- new net: R15.2, R4.1, U6.4 (FB)
- new net: C47.1, U6.6 (CB)
- new net: R22.1, R27.2, U11.1
- new net: R21.2, R22.2, U11.2 (-)
- new net: R34.1, R38.2, U13.7
- new net: R33.2, R34.2, U13.6 (-)
- new net: R4.2, R7.1
- new net: R53.2, R54.2, U15.6 (-)
- new net: C39.2, L2.1, U9.2 (SW)
- new net: R8.2, U1.1 (SD)
- new net: C33.2, L4.1, U7.2 (SW)
- new net: J1.11, R3.1, U2.6 (IO35)
- new net: R2.1, R46.2
- new net: C54.1, R37.1, U14.3 (+)
- new net: R50.1, RV3.4
- new net: C50.2, R26.1, U12.5 (+)
- new net: R39.2, R41.1, U14.2 (-)
- new net: RV3.5, U15.5 (+)
- new net: R45.2, R46.1, U9.4 (FB)
- new net: C39.1, U9.6 (CB)
- new net: R29.1, RV2.4
- new net: RV2.5, U13.5 (+)
- new net: C59.2, R54.1, U15.7
- new net: C33.1, U7.6 (CB)
- new net: C57.2, R52.1, U15.1
- new net: R51.2, R52.2, U15.2 (-)
- new net: C51.2, R28.1, U12.3 (+)
- new net: J1.10, R1.1, U2.5 (IO34)
- new net: R20.1, RV1.4
- new net +3.3VDigital: C27.1, C4.1, C6.2, U3.17 (XSMT), U3.20 (DVDD), U8.5 (OUT)
- new net +5VAnalog: C21.1, C61.1, C63.1, C65.1, C67.1, C69.1, C71.1, C73.1, C75.1, U1.4 (OUT), U1.5 (SENSE), U11.8 (V+), U12.8 (V+), U13.8 (V+), U14.8 (V+), U15.8 (V+), U16.8 (V+), U17.8 (V+), U4.8 (V+)
- new net FAHighL: R56.2, R61.2, U16.1, U16.2 (-)
- new net FAHighR: R58.2, R65.2, U16.6 (-), U16.7
- new net FALowL: C52.2, R59.2, U12.1, U12.2 (-)
- new net FALowR: C43.2, R63.2, U12.6 (-), U12.7
- new net FAMidL: R36.1, R39.1, R60.2, U14.1
- new net FAMidR: R43.1, R47.1, R64.2, U14.7
- no-connect marks 0 -> 33
Other:
- note added: "-6.5V output"
- note added: "5.5V output"
- note added: "5V output"
- note added: "RALowL - Raw Audio Low frequency Left channel RAMidL - Raw Audio Mid frequency Left channel RAHighL - Raw Audio High frequency Left channel RALowR - Raw Audio Low frequency Right channel RAMidR - Raw Audio Mid frequency Right channel RAHighR - Raw Audio High frequency Right channel FAL - Filtered Audio Left channel FAR - Filtered Audio Right channel"
- note removed: "RALowL - Raw Audio Low frequency Left channel RAMidL - Raw Audio Mid frequency Left channel RAHighL - Raw Audio High frequency Left channel RALowR - Raw Audio Low frequency Right channel RAMidR - Raw Audio Mid frequency Right channel RAHighR - Raw Audio High frequency Right channel FAL - Filtered Audio Left channel FAR - Filtered Audio Right channel +AAL - Amplified Audio Left channel Positive -A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"
- moved on the sheet: C23, C24, C25, C26, IC1, R11, R12, R13, R14, R17, R18, U4A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

Commit message: complete head unit schematic
Parts:
- added C100, C81, C82, C83, C84, C89, C90, C91, C92, C97, C98, C99: 22n, symbol Device:C_Small
- added C101, C102, C103, C104, C105, C106, C107, C108, C77, C78, C79, C80, C85, C86, C87, C88, C93, C94, C95, C96: 100n, symbol Device:C_Small
- added R100, R101, R102, R99: 7.5k, symbol Device:R_Small
- added R103, R104, R105, R106, R107, R108, R109, R110, R115, R116, R117, R118, R119, R120, R123, R124, R125, R126, R127, R128, R69, R70, R79, R80, R90, R92, R95, R96: 1k, symbol Device:R_Small
- added R111, R112: 470, symbol Device:R
- added R113, R114, R121, R122, R67, R68, R77, R78, R93, R94: 5k, symbol Device:R_Small
- added R71, R72, R81, R82, R97, R98: 500, symbol Device:R_Small
- added R73, R74, R75, R76: 16k, symbol Device:R_Small
- added R83, R84, R85, R86: 12k, symbol Device:R_Small
- added R87, R88: 56k, symbol Device:R_Small
- added R89, R91: 2k, symbol Device:R_Small
- added RV4, RV5, RV6, RV7, RV8: 10k, symbol Device:R_Potentiometer_Dual_Separate
- added U18, U19, U20, U21, U22, U23, U24, U25, U26, U27: OPA2134, AudioSystemFootprintLibrary:OPA2134UA, symbol Amplifier_Operational:OPA2134
- R21, R23, R31, R33, R51, R53: value 5k -> 1k
- R25, R26, R27, R28: value 500 -> 16k
- U11, U12, U13, U14, U15, U16, U17: footprint (none) -> AudioSystemFootprintLibrary:OPA2134UA
Connections:
- net +5VAnalog: now also J4.1 (Pin_1), C101.1, C103.1, C105.1, C107.1, C77.1, C78.1, C85.1, C86.1, C93.1, C94.1, U18.8 (V+), U19.8 (V+), U20.8 (V+), U21.8 (V+), U22.8 (V+), U23.8 (V+), U24.8 (V+), U25.8 (V+), U26.8 (V+), U27.8 (V+)
- net -5VAnalog: now also J4.2 (Pin_2), C102.1, C104.1, C106.1, C108.1, C79.1, C80.1, C87.1, C88.1, C95.1, C96.1, U18.4 (V-), U19.4 (V-), U20.4 (V-), U21.4 (V-), U22.4 (V-), U23.4 (V-), U24.4 (V-), U25.4 (V-), U26.4 (V-), U27.4 (V-)
- net FAL: now also R114.2; no longer C23.1
- net FAR: now also R113.2; no longer C24.1
- net GND: no longer J1.1, J4.8 (Pin_8)
- net GNDA: now also J1.1, U17.5 (+), U4.3 (+), U4.5 (+), C101.2, C102.2, C103.2, C104.2, C105.2, C106.2, C107.2, C108.2, C77.2, C78.2, C79.2, C80.2, C81.1, C82.1, C85.2, C86.2, C87.2, C88.2, C89.1, C90.1, C93.2, C94.2, C95.2, C96.2, R100.2, R69.1, R70.1, R79.1, R80.1, R85.2, R86.2, R90.2, R92.2, R95.1, R96.1, R99.2, RV4.3, RV4.6, RV5.3, RV5.6, RV6.3, RV6.6, RV7.3, RV7.6, RV8.3, RV8.6, U24.3 (+), U24.5 (+), U27.3 (+), U27.5 (+); no longer IC1.11 (GND2), IC1.7 (GND1), R11.1, R12.1, R13.1, R14.1, R17.1, R18.1, U17.6 (-), U4.1, U4.2 (-), U4.6 (-), U4.7
- net at C14.1, R40.2, R6.2: now also U4.6 (-), R111.1; no longer U4.5 (+)
- net at R63.1, R64.1, R65.1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: now also U17.6 (-); no longer U17.5 (+)
- net at C13.1, R44.2, R5.2: now also U4.2 (-), R112.1; no longer U4.3 (+)
- net RANCR: now reaches J3.7 (Pin_7)
- net RANCR: now also R118.1, R119.1, R120.1
- net RANCL: now reaches J3.8 (Pin_8)
- net RANCL: now also R115.1, R116.1, R117.1
- new net: R11.1, R112.2, R12.1, R13.1, U4.1
- new net: C97.2, R97.1, U22.1
- new net: R95.2, R97.2, U22.2 (-)
- new net: R124.2, R125.1, R126.1, U27.2 (-)
- new net: R123.2, R127.1, R128.1, U27.6 (-)
- new net: R128.2, U26.6 (-), U26.7
- new net: R111.2, R14.1, R17.1, R18.1, U4.7
- new net: C82.2, R76.1, U19.5 (+)
- new net: R68.1, RV4.4
- new net: R113.1, RV7.4
- new net: R79.2, R81.2, U20.2 (-)
- new net: R72.1, R74.2, U18.7
- new net: R70.2, R72.2, U18.6 (-)
- new net: RV8.5, U26.5 (+)
- new net: R126.2, U26.1, U26.2 (-)
- new net: RV8.2, U26.3 (+)
- new net: C100.1, R100.1, U23.5 (+)
- new net: C100.2, C98.1, R102.1
- new net: R103.1, R104.1, R105.1, R109.2, U24.2 (-)
- new net: C97.1, C99.2, R101.1
- new net: R121.1, RV8.4
- new net: C84.1, R74.1, R76.2
- new net: C81.2, R75.1, U19.3 (+)
- new net: R106.1, R107.1, R108.1, R110.2, U24.6 (-)
- new net: C98.2, R98.1, U22.7
- new net: R125.2, U25.1, U25.2 (-)
- new net: R96.2, R98.2, U22.6 (-)
- new net: C90.2, C92.2, R84.1, R88.2
- new net: R81.1, R83.2, U20.1
- new net: RV5.2, U20.3 (+)
- new net: R89.2, R90.1, U21.2 (-)
- new net: R71.1, R73.2, U18.1
- new net: R69.2, R71.2, U18.2 (-)
- new net: RV4.2, U18.3 (+)
- new net: RV4.5, U18.5 (+)
- new net: C89.2, C91.2, R83.1, R87.2
- new net: C91.1, R85.1, U21.3 (+)
- new net: RV6.2, U22.3 (+)
- new net: C83.1, R73.1, R75.2
- new net: R93.1, RV6.1
- new net: C99.1, R99.1, U23.3 (+)
- new net: RV5.5, U20.5 (+)
- new net: R80.2, R82.2, U20.6 (-)
- new net: R82.1, R84.2, U20.7
- new net: R77.1, RV5.1
- new net: R114.1, RV7.1
- new net: RV7.2, U25.3 (+)
- new net: R91.2, R92.1, U21.6 (-)
- new net: RV7.5, U25.5 (+)
- new net: C92.1, R86.1, U21.5 (+)
- new net: R122.1, RV8.1
- new net: R78.1, RV5.4
- new net: R94.1, RV6.4
- new net: R127.2, U25.6 (-), U25.7
- new net: R67.1, RV4.1
- new net: RV6.5, U22.5 (+)
- new net FANCHighL: R101.2, R105.2, U23.1, U23.2 (-)
- new net FANCHighR: R102.2, R108.2, U23.6 (-), U23.7
- new net FANCL: R109.1, R122.2, U24.1
- new net FANCLowL: C83.2, R103.2, U19.1, U19.2 (-)
- new net FANCLowR: C84.2, R106.2, U19.6 (-), U19.7
- new net FANCMidL: R104.2, R87.1, R89.1, U21.1
- new net FANCMidR: R107.2, R88.1, R91.1, U21.7
- new net FANCR: R110.1, R121.2, U24.7
- new net GNDPWR: IC1.11 (GND2), IC1.7 (GND1), J4.8 (Pin_8)
- new net MSL: C23.1, R124.1, U27.1
- new net MSR: C24.1, R123.1, U27.7
- new net RANCHighL: R117.2, R93.2
- new net RANCHighR: R120.2, R94.2
- new net RANCLowL: R115.2, R67.2
- new net RANCLowR: R118.2, R68.2
- new net RANCMidL: R116.2, R77.2
- new net RANCMidR: R119.2, R78.2
Other:
- note added: "R/FALowL - Raw/Filtered Audio Low frequency Left channel R/FAMidL - Raw/Filtered Audio Mid frequency Left channel R/FAHighL - Raw/Filtered Audio High frequency Left channel R/FALowR - Raw/Filtered Audio Low frequency Right channel R/FAMidR - Raw/Filtered Audio Mid frequency Right channel R/FAHighR - Raw/Filtered Audio High frequency Right channel FAL - Filtered Audio Left channel FAR - Filtered A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"
- note removed: "RALowL - Raw Audio Low frequency Left channel RAMidL - Raw Audio Mid frequency Left channel RAHighL - Raw Audio High frequency Left channel RALowR - Raw Audio Low frequency Right channel RAMidR - Raw Audio Mid frequency Right channel RAHighR - Raw Audio High frequency Right channel FAL - Filtered Audio Left channel FAR - Filtered Audio Right channel"
- moved on the sheet: C1, C10, C11, C12, C13, C14, C2, C23, C24, C25, C26, C3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

Commit message: added next/play/prev buttons (hardware and software)
Parts:
- removed C34, C35: 10u, symbol Device:C_Small
- added C34, C35: 10u, symbol Device:C_Polarized_Small_US
- added J5: Conn_02x03_Odd_Even, symbol Connector_Generic:Conn_02x03_Odd_Even
- R1, R3: value 4.7k -> 10k
- RV1, RV2, RV3, RV4, RV5, RV6, RV7, RV8: footprint (none) -> AudioSystemFootprintLibrary:PTN092H10120K1B
Connections:
- net +3.3VDigital: now also R1.2, R3.2, J5.2 (Pin_2), J5.4 (Pin_4), J5.6 (Pin_6)
- net +5VDigital: no longer R1.2, R3.2
- net GNDA: now also RV1.1, RV1.4, RV2.1, RV2.4, RV3.1, RV3.4, RV4.1, RV4.4, RV5.1, RV5.4, RV6.1, RV6.4, RV7.1, RV7.4, RV8.1, RV8.4, C34.1, C35.1; no longer RV1.3, RV1.6, RV2.3, RV2.6, RV3.3, RV3.6, RV4.3, RV4.6, RV5.3, RV5.6, RV6.3, RV6.6, RV7.3, RV7.6, RV8.3, RV8.6
- net at C31.1, C32.1, C36.1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: now also C34.2, C35.2
- net at R68.1: now also RV4.6; no longer RV4.4
- net at R113.1: now also RV7.6; no longer RV7.4
- net at R16.1: now also RV1.3; no longer RV1.1
- net at R49.1: now also RV3.3; no longer RV3.1
- net at R121.1: now also RV8.6; no longer RV8.4
- net at R30.1: now also RV2.3; no longer RV2.1
- net at R93.1: now also RV6.3; no longer RV6.1
- net at R50.1: now also RV3.6; no longer RV3.4
- net at R77.1: now also RV5.3; no longer RV5.1
- net at R114.1: now also RV7.3; no longer RV7.1
- net at R29.1: now also RV2.6; no longer RV2.4
- net at R122.1: now also RV8.3; no longer RV8.1
- net at R78.1: now also RV5.6; no longer RV5.4
- net at R94.1: now also RV6.6; no longer RV6.4
- net at R67.1: now also RV4.3; no longer RV4.1
- net at R20.1: now also RV1.6; no longer RV1.4
- net I2S_SCK: now reaches U3.13 (BCK)
- net I2S_SCK: now also U2.36 (IO22); no longer U2.10 (IO26)
- net I2S_SD: now reaches U3.14 (DIN)
- net I2S_SD: now also U2.10 (IO26); no longer U2.36 (IO22)
- net I2S_WS: now reaches U2.9 (IO25), U3.15 (LRCK)
- net AVRCP_PLAY: now reaches U2.30 (IO18)
- net AVRCP_PLAY: now also J5.3 (Pin_3)
- net AVRCP_NEXT: now reaches U2.31 (IO19)
- net AVRCP_NEXT: now also J5.5 (Pin_5)
- net AVRC_PREV: now reaches U2.33 (IO21)
- net AVRC_PREV: now also J5.1 (Pin_1)
- no-connect marks 33 -> 30
Other:
- moved on the sheet: C10, C11, C12, C13, C14, C23, C24, C25, C26, C3, C33, C36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

Commit message: added all resistor footprints
Parts:
- R1, R10, R100, R101, R102, R103, R104, R105, R106, R107, R108, R109, R11, R110, R111, R112, R113, R114, R115, R116, R117, R118, R119, R12, R120, R121, R122, R123, R124, R125, R126, R127, R128, R13, R14, R15, R16, R17, R18, R2, R20, R21, R23, R25, R26, R27, R28, R29, R3, R30, R31, R33, R35, R36, R37, R38, R39, R4, R41, R42, R43, R45, R46, R47, R48, R49, R5, R50, R51, R53, R55, R56, R57, R58, R59, R6, R60, R61, R62, R63, R64, R65, R66, R67, R68, R69, R7, R70, R73, R74, R75, R76, R77, R78, R79, R8, R80, R83, R84, R85, R86, R87, R88, R89, R9, R90, R91, R92, R93, R94, R95, R96, R99: footprint (none) -> Resistor_SMD:R_1206_3216Metric_Pad1.30x1.75mm_HandSolder
- R19: value 160 -> 180; footprint (none) -> Resistor_SMD:R_1206_3216Metric_Pad1.30x1.75mm_HandSolder
- R22, R24, R32, R34, R52, R54, R71, R72, R81, R82, R97, R98: footprint (none) -> Resistor_SMD:R_0805_2012Metric_Pad1.20x1.40mm_HandSolder
- R40, R44: value 470 -> 320; footprint (none) -> Resistor_SMD:R_1206_3216Metric_Pad1.30x1.75mm_HandSolder
Other:
- moved on the sheet: J2, J3, J4, J5
