File: Schematics/AudioSystemFull/AudioSystemFull.kicad_pcb (KiCad board)
At the start: 2 copper layers, 0 parts

Commit message: organize footprints by purpose
Parts:
- added C1: 330n, Capacitor_SMD:C_1206_3216Metric_Pad1.33x1.80mm_HandSolder, F.Cu at (551.0, 302.0)
- added C10: 0.1u, Capacitor_SMD:C_1206_3216Metric_Pad1.33x1.80mm_HandSolder, F.Cu at (541.9, 210.7)
- added C100: 22n, Capacitor_SMD:C_1206_3216Metric_Pad1.33x1.80mm_HandSolder, F.Cu at (372.4, 261.5)
- added C101: 100n, Capacitor_SMD:C_1206_3216Metric_Pad1.33x1.80mm_HandSolder, F.Cu at (317.4, 199.0)
- added C102: 100n, Capacitor_SMD:C_1206_3216Metric_Pad1.33x1.80mm_HandSolder, F.Cu at (301.9, 199.5)
- added C103: 100n, Capacitor_SMD:C_1206_3216Metric_Pad1.33x1.80mm_HandSolder, F.Cu at (466.0, 269.5)
- added C104: 100n, Capacitor_SMD:C_1206_3216Metric_Pad1.33x1.80mm_HandSolder, F.Cu at (447.9, 269.5)
- added C105: 100n, Capacitor_SMD:C_1206_3216Metric_Pad1.33x1.80mm_HandSolder, F.Cu at (496.0, 269.0)
- added C106: 100n, Capacitor_SMD:C_1206_3216Metric_Pad1.33x1.80mm_HandSolder, F.Cu at (480.0, 272.0)
- added C107: 100n, Capacitor_SMD:C_1206_3216Metric_Pad1.33x1.80mm_HandSolder, F.Cu at (480.5, 247.0)
- added C108: 100n, Capacitor_SMD:C_1206_3216Metric_Pad1.33x1.80mm_HandSolder, F.Cu at (461.5, 247.0)
- added C109: 100n, Capacitor_SMD:C_1206_3216Metric_Pad1.33x1.80mm_HandSolder, F.Cu at (546.9, 293.0)
- added C11: 10u, AudioSystemFootprintLibrary:UCZ1J100MCL1GS, F.Cu at (520.9, 198.7)
- added C110: 100n, Capacitor_SMD:C_1206_3216Metric_Pad1.33x1.80mm_HandSolder, F.Cu at (530.0, 292.0)
- added C111: 1000u, Capacitor_THT:CP_Radial_D12.5mm_P5.00mm, F.Cu at (163.5, 31.5)
- added C12: 10u, AudioSystemFootprintLibrary:UCZ1J100MCL1GS, F.Cu at (522.4, 209.7)
- added C13: 2.2n, Capacitor_SMD:C_1206_3216Metric_Pad1.33x1.80mm_HandSolder, F.Cu at (528.5, 186.0)
- added C14: 2.2n, Capacitor_SMD:C_1206_3216Metric_Pad1.33x1.80mm_HandSolder, F.Cu at (528.5, 189.3)
- added C15: 100n, Capacitor_SMD:C_1206_3216Metric_Pad1.33x1.80mm_HandSolder, F.Cu at (178.5, 61.0)
- added C16: 100n, Capacitor_SMD:C_1206_3216Metric_Pad1.33x1.80mm_HandSolder, F.Cu at (186.0, 68.5)
- added C17: 10n, Capacitor_SMD:C_1206_3216Metric_Pad1.33x1.80mm_HandSolder, F.Cu at (178.5, 66.5)
- added C18: 1u, Capacitor_SMD:C_1206_3216Metric_Pad1.33x1.80mm_HandSolder, F.Cu at (207.5, 65.5)
- added C19: 1u, Capacitor_SMD:C_1206_3216Metric_Pad1.33x1.80mm_HandSolder, F.Cu at (213.4, 65.5)
- added C2: 330n, Capacitor_SMD:C_1206_3216Metric_Pad1.33x1.80mm_HandSolder, F.Cu at (555.0, 308.0)
- added C20: 10u, AudioSystemFootprintLibrary:UCZ1J100MCL1GS, F.Cu at (212.5, 75.0)
- added C21: 10u, Capacitor_SMD:C_1206_3216Metric_Pad1.33x1.80mm_HandSolder, F.Cu at (227.5, 76.5)
- added C22: 1u, Capacitor_SMD:C_1206_3216Metric_Pad1.33x1.80mm_HandSolder, F.Cu at (212.3, 38.5)
- added C23: 220n, Capacitor_SMD:C_1206_3216Metric_Pad1.33x1.80mm_HandSolder, F.Cu at (526.5, 126.5)
- added C24: 220n, Capacitor_SMD:C_1206_3216Metric_Pad1.33x1.80mm_HandSolder, F.Cu at (533.0, 126.5)
- added C25: 100n, Capacitor_SMD:C_1206_3216Metric_Pad1.33x1.80mm_HandSolder, F.Cu at (539.5, 126.5)
- added C26: 2200u, Capacitor_THT:CP_Radial_D12.5mm_P5.00mm, F.Cu at (549.5, 122.5)
- added C27: 1u, Capacitor_SMD:C_1206_3216Metric_Pad1.33x1.80mm_HandSolder, F.Cu at (216.3, 43.0)
- added C28: 1000u, Capacitor_THT:CP_Radial_D12.5mm_P5.00mm, F.Cu at (163.0, 101.5)
- added C29: 10n, Capacitor_SMD:C_1206_3216Metric_Pad1.33x1.80mm_HandSolder, F.Cu at (179.0, 96.5)
- added C3: 10u, AudioSystemFootprintLibrary:UCZ1J100MCL1GS, F.Cu at (556.9, 200.2)
- added C30: 100n, Capacitor_SMD:C_1206_3216Metric_Pad1.33x1.80mm_HandSolder, F.Cu at (179.0, 102.0)
- added C31: 100n, Capacitor_SMD:C_1206_3216Metric_Pad1.33x1.80mm_HandSolder, F.Cu at (178.9, 107.5)
- added C32: 2.2u, Capacitor_SMD:C_1206_3216Metric_Pad1.33x1.80mm_HandSolder, F.Cu at (185.5, 103.5)
- added C33: 0.1u, Capacitor_SMD:C_1206_3216Metric_Pad1.33x1.80mm_HandSolder, F.Cu at (192.5, 107.5)
- added C34: 10u, AudioSystemFootprintLibrary:UCZ1J100MCL1GS, F.Cu at (213.0, 99.0)
- added C35: 10u, AudioSystemFootprintLibrary:UCZ1J100MCL1GS, F.Cu at (212.5, 109.0)
- added C36: 10u, Capacitor_SMD:C_1206_3216Metric_Pad1.33x1.80mm_HandSolder, F.Cu at (221.5, 96.5)
- added C37: 1000u, Capacitor_THT:CP_Radial_D12.5mm_P5.00mm, F.Cu at (164.7, 66.5)
- added C38: 2.2u, Capacitor_SMD:C_1206_3216Metric_Pad1.33x1.80mm_HandSolder, F.Cu at (179.5, 73.5)
- added C39: 0.1u, Capacitor_SMD:C_1206_3216Metric_Pad1.33x1.80mm_HandSolder, F.Cu at (192.5, 67.0)
- added C4: 10u, AudioSystemFootprintLibrary:UCZ1J100MCL1GS, F.Cu at (556.9, 210.7)
- added C40: 10u, Capacitor_SMD:C_1206_3216Metric_Pad1.33x1.80mm_HandSolder, F.Cu at (197.0, 73.5)
- added C41: 10u, Capacitor_SMD:C_1206_3216Metric_Pad1.33x1.80mm_HandSolder, F.Cu at (203.0, 73.0)
- added C42: 10u, Capacitor_SMD:C_1206_3216Metric_Pad1.33x1.80mm_HandSolder, F.Cu at (222.0, 102.5)
- added C43: 22n, Capacitor_SMD:C_1206_3216Metric_Pad1.33x1.80mm_HandSolder, F.Cu at (87.0, 252.5)
- added C44: 100n, Capacitor_SMD:C_1206_3216Metric_Pad1.33x1.80mm_HandSolder, F.Cu at (177.3, 43.0)
- added C45: 100n, Capacitor_SMD:C_1206_3216Metric_Pad1.33x1.80mm_HandSolder, F.Cu at (183.3, 43.5)
- added C46: 2.2u, Capacitor_SMD:C_1206_3216Metric_Pad1.33x1.80mm_HandSolder, F.Cu at (189.3, 45.5)
- added C47: 0.1u, Capacitor_SMD:C_1206_3216Metric_Pad1.33x1.80mm_HandSolder, F.Cu at (188.8, 39.0)
- added C48: 22u, Capacitor_SMD:C_1210_3225Metric_Pad1.33x2.70mm_HandSolder, F.Cu at (205.8, 32.0)
- added C49: 22u, Capacitor_SMD:C_1210_3225Metric_Pad1.33x2.70mm_HandSolder, F.Cu at (205.8, 36.2)
- added C5: 0.1u, Capacitor_SMD:C_1206_3216Metric_Pad1.33x1.80mm_HandSolder, F.Cu at (549.9, 193.7)
- added C50: 22n, Capacitor_SMD:C_1206_3216Metric_Pad1.33x1.80mm_HandSolder, F.Cu at (99.9, 256.5)
- added C51: 22n, Capacitor_SMD:C_1206_3216Metric_Pad1.33x1.80mm_HandSolder, F.Cu at (99.9, 251.0)
- added C52: 22n, Capacitor_SMD:C_1206_3216Metric_Pad1.33x1.80mm_HandSolder, F.Cu at (93.5, 251.0)
- added C53: 22n, Capacitor_SMD:C_1206_3216Metric_Pad1.33x1.80mm_HandSolder, F.Cu at (127.9, 259.0)
- added C54: 22n, Capacitor_SMD:C_1206_3216Metric_Pad1.33x1.80mm_HandSolder, F.Cu at (134.5, 256.5)
- added C55: 22n, Capacitor_SMD:C_1206_3216Metric_Pad1.33x1.80mm_HandSolder, F.Cu at (144.4, 257.5)
- added C56: 22n, Capacitor_SMD:C_1206_3216Metric_Pad1.33x1.80mm_HandSolder, F.Cu at (148.9, 262.5)
- added C57: 22n, Capacitor_SMD:C_1206_3216Metric_Pad1.33x1.80mm_HandSolder, F.Cu at (173.0, 262.0)
- added C58: 22n, Capacitor_SMD:C_1206_3216Metric_Pad1.33x1.80mm_HandSolder, F.Cu at (179.5, 260.5)
- added C59: 22n, Capacitor_SMD:C_1206_3216Metric_Pad1.33x1.80mm_HandSolder, F.Cu at (186.0, 260.5)
- added C6: 0.1u, Capacitor_SMD:C_1206_3216Metric_Pad1.33x1.80mm_HandSolder, F.Cu at (555.8, 191.2)
- added C60: 22n, Capacitor_SMD:C_1206_3216Metric_Pad1.33x1.80mm_HandSolder, F.Cu at (191.9, 260.5)
- added C61: 100n, Capacitor_SMD:C_1206_3216Metric_Pad1.33x1.80mm_HandSolder, F.Cu at (92.0, 283.0)
- added C62: 100n, Capacitor_SMD:C_1206_3216Metric_Pad1.33x1.80mm_HandSolder, F.Cu at (78.0, 283.5)
- added C63: 100n, Capacitor_SMD:C_1206_3216Metric_Pad1.33x1.80mm_HandSolder, F.Cu at (90.0, 242.5)
- added C64: 100n, Capacitor_SMD:C_1206_3216Metric_Pad1.33x1.80mm_HandSolder, F.Cu at (74.9, 244.5)
- added C65: 100n, Capacitor_SMD:C_1206_3216Metric_Pad1.33x1.80mm_HandSolder, F.Cu at (141.0, 276.0)
- added C66: 100n, Capacitor_SMD:C_1206_3216Metric_Pad1.33x1.80mm_HandSolder, F.Cu at (123.0, 278.0)
- added C67: 100n, Capacitor_SMD:C_1206_3216Metric_Pad1.33x1.80mm_HandSolder, F.Cu at (147.4, 242.5)
- added C68: 100n, Capacitor_SMD:C_1206_3216Metric_Pad1.33x1.80mm_HandSolder, F.Cu at (130.5, 242.5)
- added C69: 100n, Capacitor_SMD:C_1206_3216Metric_Pad1.33x1.80mm_HandSolder, F.Cu at (192.0, 244.5)
- added C7: 2.2u, Capacitor_SMD:C_1206_3216Metric_Pad1.33x1.80mm_HandSolder, F.Cu at (532.4, 200.7)
- added C70: 100n, Capacitor_SMD:C_1206_3216Metric_Pad1.33x1.80mm_HandSolder, F.Cu at (176.0, 246.0)
- added C71: 100n, Capacitor_SMD:C_1206_3216Metric_Pad1.33x1.80mm_HandSolder, F.Cu at (186.5, 273.5)
- added C72: 100n, Capacitor_SMD:C_1206_3216Metric_Pad1.33x1.80mm_HandSolder, F.Cu at (169.5, 275.0)
- added C73: 100n, Capacitor_SMD:C_1206_3216Metric_Pad1.33x1.80mm_HandSolder, F.Cu at (126.4, 204.0)
- added C74: 100n, Capacitor_SMD:C_1206_3216Metric_Pad1.33x1.80mm_HandSolder, F.Cu at (110.9, 205.5)
- added C75: 100n, Capacitor_SMD:C_1206_3216Metric_Pad1.33x1.80mm_HandSolder, F.Cu at (547.4, 249.0)
- added C76: 100n, Capacitor_SMD:C_1206_3216Metric_Pad1.33x1.80mm_HandSolder, F.Cu at (530.0, 249.5)
- added C77: 100n, Capacitor_SMD:C_1206_3216Metric_Pad1.33x1.80mm_HandSolder, F.Cu at (275.9, 251.2)
- added C78: 100n, Capacitor_SMD:C_1206_3216Metric_Pad1.33x1.80mm_HandSolder, F.Cu at (270.0, 277.8)
- added C79: 100n, Capacitor_SMD:C_1206_3216Metric_Pad1.33x1.80mm_HandSolder, F.Cu at (258.4, 252.2)
- added C8: 0.1u, Capacitor_SMD:C_1206_3216Metric_Pad1.33x1.80mm_HandSolder, F.Cu at (532.4, 205.7)
- added C80: 100n, Capacitor_SMD:C_1206_3216Metric_Pad1.33x1.80mm_HandSolder, F.Cu at (254.0, 277.8)
- added C81: 22n, Capacitor_SMD:C_1206_3216Metric_Pad1.33x1.80mm_HandSolder, F.Cu at (259.4, 260.8)
- added C82: 22n, Capacitor_SMD:C_1206_3216Metric_Pad1.33x1.80mm_HandSolder, F.Cu at (272.0, 260.8)
- added C83: 22n, Capacitor_SMD:C_1206_3216Metric_Pad1.33x1.80mm_HandSolder, F.Cu at (265.5, 260.8)
- added C84: 22n, Capacitor_SMD:C_1206_3216Metric_Pad1.33x1.80mm_HandSolder, F.Cu at (278.1, 260.8)
- added C85: 100n, Capacitor_SMD:C_1206_3216Metric_Pad1.33x1.80mm_HandSolder, F.Cu at (323.9, 243.5)
- added C86: 100n, Capacitor_SMD:C_1206_3216Metric_Pad1.33x1.80mm_HandSolder, F.Cu at (318.5, 279.5)
- added C87: 100n, Capacitor_SMD:C_1206_3216Metric_Pad1.33x1.80mm_HandSolder, F.Cu at (307.9, 244.5)
- added C88: 100n, Capacitor_SMD:C_1206_3216Metric_Pad1.33x1.80mm_HandSolder, F.Cu at (302.5, 280.0)
- added C89: 22n, Capacitor_SMD:C_1206_3216Metric_Pad1.33x1.80mm_HandSolder, F.Cu at (305.5, 258.0)
- added C9: 2.2u, Capacitor_SMD:C_1206_3216Metric_Pad1.33x1.80mm_HandSolder, F.Cu at (535.4, 210.7)
- added C90: 22n, Capacitor_SMD:C_1206_3216Metric_Pad1.33x1.80mm_HandSolder, F.Cu at (317.9, 258.0)
- added C91: 22n, Capacitor_SMD:C_1206_3216Metric_Pad1.33x1.80mm_HandSolder, F.Cu at (311.9, 258.0)
- added C92: 22n, Capacitor_SMD:C_1206_3216Metric_Pad1.33x1.80mm_HandSolder, F.Cu at (324.0, 258.0)
- added C93: 100n, Capacitor_SMD:C_1206_3216Metric_Pad1.33x1.80mm_HandSolder, F.Cu at (370.4, 275.5)
- added C94: 100n, Capacitor_SMD:C_1206_3216Metric_Pad1.33x1.80mm_HandSolder, F.Cu at (371.0, 247.0)
- added C95: 100n, Capacitor_SMD:C_1206_3216Metric_Pad1.33x1.80mm_HandSolder, F.Cu at (355.5, 275.5)
- added C96: 100n, Capacitor_SMD:C_1206_3216Metric_Pad1.33x1.80mm_HandSolder, F.Cu at (355.4, 248.0)
- added C97: 22n, Capacitor_SMD:C_1206_3216Metric_Pad1.33x1.80mm_HandSolder, F.Cu at (354.4, 261.5)
- added C98: 22n, Capacitor_SMD:C_1206_3216Metric_Pad1.33x1.80mm_HandSolder, F.Cu at (366.5, 261.5)
- added C99: 22n, Capacitor_SMD:C_1206_3216Metric_Pad1.33x1.80mm_HandSolder, F.Cu at (360.4, 261.5)
- added IC1: TDA1558Q, AudioSystemFootprintLibrary:TDA1558Q, F.Cu at (536.4, 147.4)
- added J1: SJ1-3515-SMT-TR-BE, AudioSystemFootprintLibrary:SJ1-3515-SMT-TR-BE, F.Cu at (542.5, 314.0)
- added J3: Conn_Display_Buttons, AudioSystemFootprintLibrary:Molex-43045-1211, F.Cu at (341.5, 129.6)
- added J6: Conn_ISO, AudioSystemFootprintLibrary:Conn_ISO_Solder_Pad, F.Cu at (293.9, 21.5)
- added L1: 1u, AudioSystemFootprintLibrary:SRP0315-1R0K, F.Cu at (185.8, 97.7)
- added L2: 3.3u, AudioSystemFootprintLibrary:SRP5030T-3R3M, F.Cu at (240.1, 72.0)
- added L3: 1u, AudioSystemFootprintLibrary:SRP0315-1R0K, F.Cu at (185.2, 63.2)
- added L4: 4.7u, AudioSystemFootprintLibrary:VLS6045EX-4R7M-H, F.Cu at (195.5, 100.0)
- added L6: 1u, AudioSystemFootprintLibrary:SRP0315-1R0K, F.Cu at (180.6, 36.2)
- added L7: 10u, AudioSystemFootprintLibrary:SRR1280A-100M, F.Cu at (193.3, 27.0)
- added R1: 10k, Resistor_SMD:R_1206_3216Metric_Pad1.30x1.75mm_HandSolder, F.Cu at (554.0, 314.0)
- added R10: 100k, Resistor_SMD:R_1206_3216Metric_Pad1.30x1.75mm_HandSolder, F.Cu at (204.0, 98.0)
- added R100: 7.5k, Resistor_SMD:R_1206_3216Metric_Pad1.30x1.75mm_HandSolder, F.Cu at (366.5, 255.5)
- added R101: 7.5k, Resistor_SMD:R_1206_3216Metric_Pad1.30x1.75mm_HandSolder, F.Cu at (360.5, 255.5)
- added R102: 7.5k, Resistor_SMD:R_1206_3216Metric_Pad1.30x1.75mm_HandSolder, F.Cu at (372.5, 255.5)
- added R103: 1k, Resistor_SMD:R_1206_3216Metric_Pad1.30x1.75mm_HandSolder, F.Cu at (301.0, 213.5)
- added R104: 1k, Resistor_SMD:R_1206_3216Metric_Pad1.30x1.75mm_HandSolder, F.Cu at (308.5, 213.5)
- added R105: 1k, Resistor_SMD:R_1206_3216Metric_Pad1.30x1.75mm_HandSolder, F.Cu at (314.5, 213.5)
- added R106: 1k, Resistor_SMD:R_1206_3216Metric_Pad1.30x1.75mm_HandSolder, F.Cu at (300.9, 207.5)
- added R107: 1k, Resistor_SMD:R_1206_3216Metric_Pad1.30x1.75mm_HandSolder, F.Cu at (307.4, 207.5)
- added R108: 1k, Resistor_SMD:R_1206_3216Metric_Pad1.30x1.75mm_HandSolder, F.Cu at (313.5, 207.5)
- added R109: 1k, Resistor_SMD:R_1206_3216Metric_Pad1.30x1.75mm_HandSolder, F.Cu at (320.5, 213.5)
- added R11: 1k, Resistor_SMD:R_1206_3216Metric_Pad1.30x1.75mm_HandSolder, F.Cu at (528.0, 236.7)
- added R110: 1k, Resistor_SMD:R_1206_3216Metric_Pad1.30x1.75mm_HandSolder, F.Cu at (319.5, 207.5)
- added R111: 470, Resistor_SMD:R_1206_3216Metric_Pad1.30x1.75mm_HandSolder, F.Cu at (542.0, 242.5)
- added R112: 470, Resistor_SMD:R_1206_3216Metric_Pad1.30x1.75mm_HandSolder, F.Cu at (535.5, 242.5)
- added R113: 5k, Resistor_SMD:R_1206_3216Metric_Pad1.30x1.75mm_HandSolder, F.Cu at (461.4, 280.5)
- added R114: 5k, Resistor_SMD:R_1206_3216Metric_Pad1.30x1.75mm_HandSolder, F.Cu at (454.5, 280.5)
- added R115: 1k, Resistor_SMD:R_1206_3216Metric_Pad1.30x1.75mm_HandSolder, F.Cu at (268.4, 226.7)
- added R116: 1k, Resistor_SMD:R_1206_3216Metric_Pad1.30x1.75mm_HandSolder, F.Cu at (268.4, 230.0)
- added R117: 1k, Resistor_SMD:R_1206_3216Metric_Pad1.30x1.75mm_HandSolder, F.Cu at (277.0, 220.5)
- added R118: 1k, Resistor_SMD:R_1206_3216Metric_Pad1.30x1.75mm_HandSolder, F.Cu at (277.0, 223.8)
- added R119: 1k, Resistor_SMD:R_1206_3216Metric_Pad1.30x1.75mm_HandSolder, F.Cu at (277.0, 227.1)
- added R12: 1k, Resistor_SMD:R_1206_3216Metric_Pad1.30x1.75mm_HandSolder, F.Cu at (528.0, 240.0)
- added R120: 1k, Resistor_SMD:R_1206_3216Metric_Pad1.30x1.75mm_HandSolder, F.Cu at (277.0, 230.4)
- added R121: 5k, Resistor_SMD:R_1206_3216Metric_Pad1.30x1.75mm_HandSolder, F.Cu at (485.0, 280.0)
- added R122: 5k, Resistor_SMD:R_1206_3216Metric_Pad1.30x1.75mm_HandSolder, F.Cu at (491.4, 280.0)
- added R123: 1k, Resistor_SMD:R_1206_3216Metric_Pad1.30x1.75mm_HandSolder, F.Cu at (477.1, 241.0)
- added R124: 1k, Resistor_SMD:R_1206_3216Metric_Pad1.30x1.75mm_HandSolder, F.Cu at (465.5, 241.5)
- added R125: 1k, Resistor_SMD:R_1206_3216Metric_Pad1.30x1.75mm_HandSolder, F.Cu at (461.5, 262.5)
- added R126: 1k, Resistor_SMD:R_1206_3216Metric_Pad1.30x1.75mm_HandSolder, F.Cu at (482.0, 262.0)
- added R127: 1k, Resistor_SMD:R_1206_3216Metric_Pad1.30x1.75mm_HandSolder, F.Cu at (454.5, 262.0)
- added R128: 1k, Resistor_SMD:R_1206_3216Metric_Pad1.30x1.75mm_HandSolder, F.Cu at (490.0, 262.0)
- added R13: 1k, Resistor_SMD:R_1206_3216Metric_Pad1.30x1.75mm_HandSolder, F.Cu at (528.0, 243.3)
- added R14: 1k, Resistor_SMD:R_1206_3216Metric_Pad1.30x1.75mm_HandSolder, F.Cu at (549.0, 233.5)
- added R15: 100k, Resistor_SMD:R_1206_3216Metric_Pad1.30x1.75mm_HandSolder, F.Cu at (195.8, 39.0)
- added R16: 5k, Resistor_SMD:R_1206_3216Metric_Pad1.30x1.75mm_HandSolder, F.Cu at (83.0, 266.0)
- added R17: 1k, Resistor_SMD:R_1206_3216Metric_Pad1.30x1.75mm_HandSolder, F.Cu at (549.0, 238.0)
- added R18: 1k, Resistor_SMD:R_1206_3216Metric_Pad1.30x1.75mm_HandSolder, F.Cu at (549.0, 243.0)
- added R19: 180, Resistor_SMD:R_1206_3216Metric_Pad1.30x1.75mm_HandSolder, F.Cu at (199.5, 107.5)
- added R2: 240, Resistor_SMD:R_1206_3216Metric_Pad1.30x1.75mm_HandSolder, F.Cu at (199.5, 67.0)
- added R20: 5k, Resistor_SMD:R_1206_3216Metric_Pad1.30x1.75mm_HandSolder, F.Cu at (83.0, 271.0)
- added R21: 1k, Resistor_SMD:R_1206_3216Metric_Pad1.30x1.75mm_HandSolder, F.Cu at (93.0, 277.0)
- added R22: 500, Resistor_SMD:R_0805_2012Metric_Pad1.20x1.40mm_HandSolder, F.Cu at (90.5, 270.0)
- added R23: 1k, Resistor_SMD:R_1206_3216Metric_Pad1.30x1.75mm_HandSolder, F.Cu at (95.5, 269.5)
- added R24: 500, Resistor_SMD:R_0805_2012Metric_Pad1.20x1.40mm_HandSolder, F.Cu at (90.5, 265.0)
- added R25: 16k, Resistor_SMD:R_1206_3216Metric_Pad1.30x1.75mm_HandSolder, F.Cu at (87.0, 260.0)
- added R26: 16k, Resistor_SMD:R_1206_3216Metric_Pad1.30x1.75mm_HandSolder, F.Cu at (94.0, 260.0)
- added R27: 16k, Resistor_SMD:R_1206_3216Metric_Pad1.30x1.75mm_HandSolder, F.Cu at (101.0, 262.0)
- added R28: 16k, Resistor_SMD:R_1206_3216Metric_Pad1.30x1.75mm_HandSolder, F.Cu at (102.0, 267.5)
- added R29: 5k, Resistor_SMD:R_1206_3216Metric_Pad1.30x1.75mm_HandSolder, F.Cu at (136.5, 283.0)
- added R3: 10k, Resistor_SMD:R_1206_3216Metric_Pad1.30x1.75mm_HandSolder, F.Cu at (558.0, 319.0)
- added R30: 5k, Resistor_SMD:R_1206_3216Metric_Pad1.30x1.75mm_HandSolder, F.Cu at (130.5, 284.5)
- added R31: 1k, Resistor_SMD:R_1206_3216Metric_Pad1.30x1.75mm_HandSolder, F.Cu at (126.0, 271.5)
- added R32: 500, Resistor_SMD:R_0805_2012Metric_Pad1.20x1.40mm_HandSolder, F.Cu at (131.0, 269.0)
- added R33: 1k, Resistor_SMD:R_1206_3216Metric_Pad1.30x1.75mm_HandSolder, F.Cu at (135.9, 269.0)
- added R34: 500, Resistor_SMD:R_0805_2012Metric_Pad1.20x1.40mm_HandSolder, F.Cu at (141.5, 270.5)
- added R35: 12k, Resistor_SMD:R_1206_3216Metric_Pad1.30x1.75mm_HandSolder, F.Cu at (133.9, 262.5)
- added R36: 56k, Resistor_SMD:R_1206_3216Metric_Pad1.30x1.75mm_HandSolder, F.Cu at (128.9, 252.0)
- added R37: 12k, Resistor_SMD:R_1206_3216Metric_Pad1.30x1.75mm_HandSolder, F.Cu at (135.5, 250.0)
- added R38: 12k, Resistor_SMD:R_1206_3216Metric_Pad1.30x1.75mm_HandSolder, F.Cu at (142.4, 264.0)
- added R39: 2k, Resistor_SMD:R_1206_3216Metric_Pad1.30x1.75mm_HandSolder, F.Cu at (141.9, 237.5)
- added R4: 11k, Resistor_SMD:R_1206_3216Metric_Pad1.30x1.75mm_HandSolder, F.Cu at (202.3, 42.5)
- added R40: 320, Resistor_SMD:R_1206_3216Metric_Pad1.30x1.75mm_HandSolder, F.Cu at (540.0, 287.0)
- added R41: 1k, Resistor_SMD:R_1206_3216Metric_Pad1.30x1.75mm_HandSolder, F.Cu at (134.5, 236.5)
- added R42: 12k, Resistor_SMD:R_1206_3216Metric_Pad1.30x1.75mm_HandSolder, F.Cu at (145.0, 249.0)
- added R43: 56k, Resistor_SMD:R_1206_3216Metric_Pad1.30x1.75mm_HandSolder, F.Cu at (149.9, 253.0)
- added R44: 320, Resistor_SMD:R_1206_3216Metric_Pad1.30x1.75mm_HandSolder, F.Cu at (533.0, 284.5)
- added R45: 100k, Resistor_SMD:R_1206_3216Metric_Pad1.30x1.75mm_HandSolder, F.Cu at (193.0, 61.5)
- added R46: 12k, Resistor_SMD:R_1206_3216Metric_Pad1.30x1.75mm_HandSolder, F.Cu at (200.0, 61.5)
- added R47: 2k, Resistor_SMD:R_1206_3216Metric_Pad1.30x1.75mm_HandSolder, F.Cu at (148.6, 237.5)
- added R48: 1k, Resistor_SMD:R_1206_3216Metric_Pad1.30x1.75mm_HandSolder, F.Cu at (142.0, 232.0)
- added R49: 5k, Resistor_SMD:R_1206_3216Metric_Pad1.30x1.75mm_HandSolder, F.Cu at (177.9, 282.0)
- added R5: 470, Resistor_SMD:R_1206_3216Metric_Pad1.30x1.75mm_HandSolder, F.Cu at (538.0, 189.0)
- added R50: 5k, Resistor_SMD:R_1206_3216Metric_Pad1.30x1.75mm_HandSolder, F.Cu at (184.5, 282.0)
- added R51: 1k, Resistor_SMD:R_1206_3216Metric_Pad1.30x1.75mm_HandSolder, F.Cu at (178.5, 266.5)
- added R52: 500, Resistor_SMD:R_0805_2012Metric_Pad1.20x1.40mm_HandSolder, F.Cu at (184.0, 267.0)
- added R53: 1k, Resistor_SMD:R_1206_3216Metric_Pad1.30x1.75mm_HandSolder, F.Cu at (190.0, 267.0)
- added R54: 500, Resistor_SMD:R_0805_2012Metric_Pad1.20x1.40mm_HandSolder, F.Cu at (196.0, 267.0)
- added R55: 7.5k, Resistor_SMD:R_1206_3216Metric_Pad1.30x1.75mm_HandSolder, F.Cu at (175.5, 254.5)
- added R56: 7.5k, Resistor_SMD:R_1206_3216Metric_Pad1.30x1.75mm_HandSolder, F.Cu at (181.4, 254.5)
- added R57: 7.5k, Resistor_SMD:R_1206_3216Metric_Pad1.30x1.75mm_HandSolder, F.Cu at (187.4, 254.5)
- added R58: 7.5k, Resistor_SMD:R_1206_3216Metric_Pad1.30x1.75mm_HandSolder, F.Cu at (193.9, 254.5)
- added R59: 1k, Resistor_SMD:R_1206_3216Metric_Pad1.30x1.75mm_HandSolder, F.Cu at (109.5, 219.5)
- added R6: 470, Resistor_SMD:R_1206_3216Metric_Pad1.30x1.75mm_HandSolder, F.Cu at (538.0, 192.3)
- added R60: 1k, Resistor_SMD:R_1206_3216Metric_Pad1.30x1.75mm_HandSolder, F.Cu at (115.5, 219.5)
- added R61: 1k, Resistor_SMD:R_1206_3216Metric_Pad1.30x1.75mm_HandSolder, F.Cu at (121.5, 219.5)
- added R62: 1k, Resistor_SMD:R_1206_3216Metric_Pad1.30x1.75mm_HandSolder, F.Cu at (128.0, 219.5)
- added R63: 1k, Resistor_SMD:R_1206_3216Metric_Pad1.30x1.75mm_HandSolder, F.Cu at (109.0, 212.5)
- added R64: 1k, Resistor_SMD:R_1206_3216Metric_Pad1.30x1.75mm_HandSolder, F.Cu at (115.5, 212.5)
- added R65: 1k, Resistor_SMD:R_1206_3216Metric_Pad1.30x1.75mm_HandSolder, F.Cu at (122.0, 212.5)
- added R66: 1k, Resistor_SMD:R_1206_3216Metric_Pad1.30x1.75mm_HandSolder, F.Cu at (128.0, 212.5)
- added R67: 5k, Resistor_SMD:R_1206_3216Metric_Pad1.30x1.75mm_HandSolder, F.Cu at (259.4, 284.2)
- added R68: 5k, Resistor_SMD:R_1206_3216Metric_Pad1.30x1.75mm_HandSolder, F.Cu at (265.5, 284.2)
- added R69: 1k, Resistor_SMD:R_1206_3216Metric_Pad1.30x1.75mm_HandSolder, F.Cu at (259.0, 271.2)
- added R7: 2.7k, Resistor_SMD:R_1206_3216Metric_Pad1.30x1.75mm_HandSolder, F.Cu at (196.8, 46.0)
- added R70: 1k, Resistor_SMD:R_1206_3216Metric_Pad1.30x1.75mm_HandSolder, F.Cu at (270.0, 271.2)
- added R71: 500, Resistor_SMD:R_0805_2012Metric_Pad1.20x1.40mm_HandSolder, F.Cu at (264.5, 271.2)
- added R72: 500, Resistor_SMD:R_0805_2012Metric_Pad1.20x1.40mm_HandSolder, F.Cu at (275.5, 271.2)
- added R73: 16k, Resistor_SMD:R_1206_3216Metric_Pad1.30x1.75mm_HandSolder, F.Cu at (253.5, 266.2)
- added R74: 16k, Resistor_SMD:R_1206_3216Metric_Pad1.30x1.75mm_HandSolder, F.Cu at (265.0, 266.2)
- added R75: 16k, Resistor_SMD:R_1206_3216Metric_Pad1.30x1.75mm_HandSolder, F.Cu at (259.5, 266.2)
- added R76: 16k, Resistor_SMD:R_1206_3216Metric_Pad1.30x1.75mm_HandSolder, F.Cu at (271.0, 266.2)
- added R77: 5k, Resistor_SMD:R_1206_3216Metric_Pad1.30x1.75mm_HandSolder, F.Cu at (309.4, 286.0)
- added R78: 5k, Resistor_SMD:R_1206_3216Metric_Pad1.30x1.75mm_HandSolder, F.Cu at (314.9, 286.0)
- added R79: 1k, Resistor_SMD:R_1206_3216Metric_Pad1.30x1.75mm_HandSolder, F.Cu at (305.0, 272.0)
- added R8: 10k, Resistor_SMD:R_1206_3216Metric_Pad1.30x1.75mm_HandSolder, F.Cu at (221.5, 76.5)
- added R80: 1k, Resistor_SMD:R_1206_3216Metric_Pad1.30x1.75mm_HandSolder, F.Cu at (316.0, 272.0)
- added R81: 500, Resistor_SMD:R_0805_2012Metric_Pad1.20x1.40mm_HandSolder, F.Cu at (310.5, 272.0)
- added R82: 500, Resistor_SMD:R_0805_2012Metric_Pad1.20x1.40mm_HandSolder, F.Cu at (321.5, 272.0)
- added R83: 12k, Resistor_SMD:R_1206_3216Metric_Pad1.30x1.75mm_HandSolder, F.Cu at (305.9, 264.0)
- added R84: 12k, Resistor_SMD:R_1206_3216Metric_Pad1.30x1.75mm_HandSolder, F.Cu at (311.5, 264.0)
- added R85: 12k, Resistor_SMD:R_1206_3216Metric_Pad1.30x1.75mm_HandSolder, F.Cu at (305.5, 252.5)
- added R86: 12k, Resistor_SMD:R_1206_3216Metric_Pad1.30x1.75mm_HandSolder, F.Cu at (317.5, 252.5)
- added R87: 56k, Resistor_SMD:R_1206_3216Metric_Pad1.30x1.75mm_HandSolder, F.Cu at (311.5, 252.5)
- added R88: 56k, Resistor_SMD:R_1206_3216Metric_Pad1.30x1.75mm_HandSolder, F.Cu at (324.0, 252.5)
- added R89: 2k, Resistor_SMD:R_1206_3216Metric_Pad1.30x1.75mm_HandSolder, F.Cu at (305.0, 235.5)
- added R9: 10k, Resistor_SMD:R_1206_3216Metric_Pad1.30x1.75mm_HandSolder, F.Cu at (204.4, 103.5)
- added R90: 1k, Resistor_SMD:R_1206_3216Metric_Pad1.30x1.75mm_HandSolder, F.Cu at (311.0, 235.5)
- added R91: 2k, Resistor_SMD:R_1206_3216Metric_Pad1.30x1.75mm_HandSolder, F.Cu at (317.0, 235.5)
- added R92: 1k, Resistor_SMD:R_1206_3216Metric_Pad1.30x1.75mm_HandSolder, F.Cu at (323.4, 235.5)
- added R93: 5k, Resistor_SMD:R_1206_3216Metric_Pad1.30x1.75mm_HandSolder, F.Cu at (360.9, 284.5)
- added R94: 5k, Resistor_SMD:R_1206_3216Metric_Pad1.30x1.75mm_HandSolder, F.Cu at (367.0, 284.5)
- added R95: 1k, Resistor_SMD:R_1206_3216Metric_Pad1.30x1.75mm_HandSolder, F.Cu at (355.0, 267.5)
- added R96: 1k, Resistor_SMD:R_1206_3216Metric_Pad1.30x1.75mm_HandSolder, F.Cu at (366.5, 267.5)
- added R97: 500, Resistor_SMD:R_0805_2012Metric_Pad1.20x1.40mm_HandSolder, F.Cu at (361.0, 267.5)
- added R98: 500, Resistor_SMD:R_0805_2012Metric_Pad1.20x1.40mm_HandSolder, F.Cu at (372.0, 267.5)
- added R99: 7.5k, Resistor_SMD:R_1206_3216Metric_Pad1.30x1.75mm_HandSolder, F.Cu at (354.0, 255.5)
- added RV1: 10k, AudioSystemFootprintLibrary:PTN092H10120K1B, F.Cu at (82.1, 289.2)
- added RV2: 10k, AudioSystemFootprintLibrary:PTN092H10120K1B, F.Cu at (131.5, 289.8)
- added RV3: 10k, AudioSystemFootprintLibrary:PTN092H10120K1B, F.Cu at (180.0, 290.5)
- added RV4: 10k, AudioSystemFootprintLibrary:PTN092H10120K1B, F.Cu at (262.5, 292.8)
- added RV5: 10k, AudioSystemFootprintLibrary:PTN092H10120K1B, F.Cu at (310.5, 292.2)
- added RV6: 10k, AudioSystemFootprintLibrary:PTN092H10120K1B, F.Cu at (361.0, 292.0)
- added RV7: 10k, AudioSystemFootprintLibrary:PTN092H10120K1B, F.Cu at (460.0, 287.5)
- added RV8: 10k, AudioSystemFootprintLibrary:PTN092H10120K1B, F.Cu at (485.2, 288.0)
- added U1: LP3856ES-5.0, AudioSystemFootprintLibrary:LP3856ES-5.0, F.Cu at (226.5, 65.7)
- added U10: LT3015EQ-5PBF, AudioSystemFootprintLibrary:LT3015EQ-5PBF, F.Cu at (232.5, 102.5)
- added U11: OPA2134, AudioSystemFootprintLibrary:OPA2134UA, F.Cu at (85.0, 281.5)
- added U12: OPA2134, AudioSystemFootprintLibrary:OPA2134UA, F.Cu at (83.0, 244.5)
- added U13: OPA2134, AudioSystemFootprintLibrary:OPA2134UA, F.Cu at (131.5, 276.5)
- added U14: OPA2134, AudioSystemFootprintLibrary:OPA2134UA, F.Cu at (139.5, 244.0)
- added U15: OPA2134, AudioSystemFootprintLibrary:OPA2134UA, F.Cu at (179.0, 274.0)
- added U16: OPA2134, AudioSystemFootprintLibrary:OPA2134UA, F.Cu at (184.0, 246.5)
- added U17: OPA2134, AudioSystemFootprintLibrary:OPA2134UA, F.Cu at (118.5, 204.5)
- added U18: OPA2134, AudioSystemFootprintLibrary:OPA2134UA, F.Cu at (262.5, 277.8)
- added U19: OPA2134, AudioSystemFootprintLibrary:OPA2134UA, F.Cu at (268.0, 251.8)
- added U2: DEVKIT_V1_ESP32-WROOM-32, AudioSystemFootprintLibrary:MODULE_DEVKIT_V1_ESP32-WROOM-32, F.Cu at (343.0, 101.5)
- added U20: OPA2134, AudioSystemFootprintLibrary:OPA2134UA, F.Cu at (310.5, 279.9)
- added U21: OPA2134, AudioSystemFootprintLibrary:OPA2134UA, F.Cu at (316.0, 244.1)
- added U22: OPA2134, AudioSystemFootprintLibrary:OPA2134UA, F.Cu at (363.0, 276.0)
- added U23: OPA2134, AudioSystemFootprintLibrary:OPA2134UA, F.Cu at (363.5, 247.6)
- added U24: OPA2134, AudioSystemFootprintLibrary:OPA2134UA, F.Cu at (310.0, 199.5)
- added U25: OPA2134, AudioSystemFootprintLibrary:OPA2134UA, F.Cu at (457.5, 271.0)
- added U26: OPA2134, AudioSystemFootprintLibrary:OPA2134UA, F.Cu at (487.0, 270.0)
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
Commit message: footprint placement part 1
Parts:
- C11, C12, C3, C4: footprint AudioSystemFootprintLibrary:UCZ1J100MCL1GS -> Capacitor_SMD:C_1206_3216Metric_Pad1.33x1.80mm_HandSolder
- moved R3 408.1 mm to (175.4, 176.8)
- moved C1 408.1 mm to (168.5, 159.8)
- moved C2 408.1 mm to (172.5, 165.8)
- moved J1 408.1 mm to (160.0, 171.8)
- moved R1 408.1 mm to (171.5, 171.8)
- moved C109 359.2 mm to (199.0, 203.6)
- moved U28 357.3 mm to (192.6, 205.8)
- moved R44 356.4 mm to (185.8, 204.0), turned to 180 degrees
- moved C110 354.0 mm to (186.2, 207.8), turned to 180 degrees
- moved R40 350.5 mm to (199.0, 206.0)
- moved C4 341.3 mm to (220.0, 155.6)
- moved C6 337.4 mm to (220.0, 158.2), turned to 180 degrees
- moved C3 334.6 mm to (225.2, 155.6), turned to 180 degrees
- moved C5 326.6 mm to (225.2, 158.2), turned to 180 degrees
- moved C10 326.3 mm to (218.0, 170.8), turned to 90 degrees
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Connections:
- U1 pad 6: (no net) -> GNDA
Routing:
- net +3.3VAnalog: track 0.00 -> 0.84 mm
Other:
- copper layers 2 -> 4
- board text added: "+"

Commit message: footprint placement possibly done, minor schematic changes
Parts:
- added R129: 0, Resistor_SMD:R_0805_2012Metric_Pad1.20x1.40mm_HandSolder, F.Cu at (313.1, 212.4)
- added R130: 0, Resistor_SMD:R_0805_2012Metric_Pad1.20x1.40mm_HandSolder, F.Cu at (280.7, 213.7)
- added R131: 0, Resistor_SMD:R_0805_2012Metric_Pad1.20x1.40mm_HandSolder, F.Cu at (310.3, 197.8)
- added R132: 0, Resistor_SMD:R_0805_2012Metric_Pad1.20x1.40mm_HandSolder, F.Cu at (342.7, 197.3)
- added R133: 0, Resistor_SMD:R_0805_2012Metric_Pad1.20x1.40mm_HandSolder, F.Cu at (277.9, 198.4)
- C1, C10, C100, C101, C102, C103, C104, C105, C106, C107, C108, C109, C110, C13, C14, C15, C16, C17, C18, C19, C2, C21, C22, C23, C24, C25, C27, C29, C30, C31, C32, C33, C36, C38, C39, C40, C41, C42, C43, C44, C45, C46, C47, C5, C50, C51, C52, C53, C54, C55, C56, C57, C58, C59, C6, C60, C61, C62, C63, C64, C65, C66, C67, C68, C69, C7, C70, C71, C72, C73, C74, C75, C76, C77, C78, C79, C8, C80, C81, C82, C83, C84, C85, C86, C87, C88, C89, C9, C90, C91, C92, C93, C94, C95, C96, C97, C98, C99: footprint Capacitor_SMD:C_1206_3216Metric_Pad1.33x1.80mm_HandSolder -> Capacitor_SMD:C_0805_2012Metric_Pad1.18x1.45mm_HandSolder
- C20, C34, C35: footprint AudioSystemFootprintLibrary:UCZ1J100MCL1GS -> Capacitor_SMD:C_0805_2012Metric_Pad1.18x1.45mm_HandSolder
- C48, C49: value 22u -> 10u; footprint Capacitor_SMD:C_1210_3225Metric_Pad1.33x2.70mm_HandSolder -> Capacitor_SMD:C_0805_2012Metric_Pad1.18x1.45mm_HandSolder
- L2: value 3.3u -> 4.7u; footprint AudioSystemFootprintLibrary:SRP5030T-3R3M -> AudioSystemFootprintLibrary:VLS6045EX-4R7M-H
- L7: value 10u -> 4.7u; footprint AudioSystemFootprintLibrary:SRR1280A-100M -> AudioSystemFootprintLibrary:VLS6045EX-4R7M-H
- R1, R10, R100, R101, R102, R103, R104, R105, R106, R107, R108, R109, R11, R110, R111, R112, R113, R114, R115, R116, R117, R118, R119, R12, R120, R121, R122, R123, R124, R125, R126, R127, R128, R13, R14, R15, R16, R17, R18, R2, R20, R21, R23, R25, R26, R27, R28, R29, R3, R30, R31, R33, R35, R36, R37, R38, R39, R4, R40, R41, R42, R43, R44, R45, R46, R47, R48, R49, R5, R50, R51, R53, R55, R56, R57, R58, R59, R6, R60, R61, R62, R63, R64, R65, R66, R67, R68, R69, R7, R70, R73, R74, R75, R76, R77, R78, R79, R80, R83, R84, R85, R86, R87, R88, R89, R90, R91, R92, R93, R94, R95, R96, R99: footprint Resistor_SMD:R_1206_3216Metric_Pad1.30x1.75mm_HandSolder -> Resistor_SMD:R_0805_2012Metric_Pad1.20x1.40mm_HandSolder
- R19: value 180 -> 110; footprint Resistor_SMD:R_1206_3216Metric_Pad1.30x1.75mm_HandSolder -> Resistor_SMD:R_0805_2012Metric_Pad1.20x1.40mm_HandSolder
- R8: value 10k -> 0; footprint Resistor_SMD:R_1206_3216Metric_Pad1.30x1.75mm_HandSolder -> Resistor_SMD:R_0805_2012Metric_Pad1.20x1.40mm_HandSolder
- R9: value 10k -> 11k; footprint Resistor_SMD:R_1206_3216Metric_Pad1.30x1.75mm_HandSolder -> Resistor_SMD:R_0805_2012Metric_Pad1.20x1.40mm_HandSolder
- U1: value LP3856ES-5.0 -> MIC39100-5.0WS; footprint AudioSystemFootprintLibrary:LP3856ES-5.0 -> AudioSystemFootprintLibrary:MIC39100-5.0WS
- U6: value LMR51420XFDDCR -> LMR51420YFDDCR; footprint AudioSystemFootprintLibrary:LMR51420XFDDCR -> AudioSystemFootprintLibrary:LMR51420YFDDCR
- U9: value LMR51430YFDDCR -> LMR51420YFDDCR; footprint AudioSystemFootprintLibrary:LMR51430YFDDCR -> AudioSystemFootprintLibrary:LMR51420YFDDCR
- moved C42 270.8 mm to (344.3, 212.8), turned to -90 degrees
- moved R9 262.0 mm to (335.9, 203.7)
- moved C34 261.9 mm to (350.4, 211.5), turned to 0 degrees
- moved R10 261.7 mm to (338.1, 203.7)
- moved R19 261.5 mm to (335.9, 207.7)
- moved C32 261.2 mm to (341.7, 200.9)
- moved C30 261.2 mm to (338.0, 197.3), turned to -90 degrees
- moved L4 261.0 mm to (348.9, 206.1)
- moved C33 260.9 mm to (341.4, 206.7)
- moved U7 260.5 mm to (341.5, 203.8)
- moved C29 260.5 mm to (335.8, 197.3), turned to -90 degrees
- moved C35 259.9 mm to (350.4, 213.7), turned to 0 degrees
- moved C31 259.8 mm to (340.5, 197.3), turned to -90 degrees
- moved L1 257.1 mm to (339.3, 192.5), turned to 0 degrees
- moved C36 256.0 mm to (345.2, 216.7), turned to -90 degrees
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Connections:
- C111 pad 2: GNDA -> GNDPWR
- C15 pad 2: GNDA -> GNDPWR
- C16 pad 1: Net-(U9-EN) -> Net-(C16-Pad1)
- C16 pad 2: GNDA -> GNDPWR
- C17 pad 2: GNDA -> GNDPWR
- C28 pad 2: GNDA -> GNDPWR
- C29 pad 2: GNDA -> GNDPWR
- C30 pad 2: GNDA -> GNDPWR
- C31 pad 1: Net-(U10-*SHDN) -> Net-(C31-Pad1)
- C31 pad 2: GNDA -> GNDPWR
- C32 pad 1: Net-(U10-*SHDN) -> Net-(U7-GND)
- C34 pad 1: GNDA -> Net-(U7-GND)
- C34 pad 2: Net-(U10-*SHDN) -> GNDA
- C35 pad 1: GNDA -> Net-(U7-GND)
- C35 pad 2: Net-(U10-*SHDN) -> GNDA
- C37 pad 2: GNDA -> GNDPWR
- C40 pad 1: Net-(U1-IN) -> Net-(C40-Pad1)
- C41 pad 1: Net-(U1-IN) -> Net-(C40-Pad1)
- C44 pad 2: GND -> GNDPWR
- C45 pad 1: Net-(U6-EN) -> Net-(C45-Pad1)
- C45 pad 2: GND -> GNDPWR
- C48 pad 1: +5VDigital -> Net-(C48-Pad1)
- C49 pad 1: +5VDigital -> Net-(C48-Pad1)
- J6 pad a3: unconnected-(J6-Pin_a3-Pada3) -> GNDA
- L1 pad 2: Net-(U10-*SHDN) -> Net-(C31-Pad1)
- L2 pad 2: Net-(U1-IN) -> Net-(C40-Pad1)
- L3 pad 2: Net-(U9-EN) -> Net-(C16-Pad1)
- L6 pad 2: Net-(U6-EN) -> Net-(C45-Pad1)
- L7 pad 2: +5VDigital -> Net-(C48-Pad1)
- R10 pad 2: Net-(U10-*SHDN) -> Net-(U7-GND)
- R15 pad 1: +5VDigital -> Net-(C48-Pad1)
- R45 pad 1: Net-(U1-IN) -> Net-(C40-Pad1)
- R8 pad 1: Net-(U1-IN) -> Net-(U7-GND)
- R8 pad 2: Net-(U1-SD) -> Net-(U10-*SHDN)
- U1 pad 1: Net-(U1-SD) -> Net-(U1-IN)
- U1 pad 2: Net-(U1-IN) -> GNDA
- U1 pad 3: GNDA -> +5VAnalog
- U7 pad 1: Net-(U10-*SHDN) -> Net-(U7-GND)
- U7 pad 3: Net-(U10-*SHDN) -> Net-(U7-GND)
Other:
- board outline added: 232.1 x 165.8 mm
- copper layers 4 -> 2

Commit message: progress sync
Parts:
- added G***: LOGO, LOGO, F.Cu at (174.6, 166.2)
- added G***: LOGO, LOGO, F.Cu at (214.1, 159.1)
- C11, C12, C3, C4: footprint Capacitor_SMD:C_1206_3216Metric_Pad1.33x1.80mm_HandSolder -> Capacitor_SMD:C_0805_2012Metric_Pad1.18x1.45mm_HandSolder
- moved R3 28.5 mm to (195.2, 215.3), turned to -90 degrees
- moved R1 25.3 mm to (193.0, 215.3), turned to -90 degrees
- moved U2 14.1 mm to (203.1, 198.3)
- moved J6 12.1 mm to (327.7, 185.2)
- moved J3 5.33 mm to (249.1, 218.9)
- moved R118 3.57 mm to (298.7, 241.4)
- moved R120 3.57 mm to (302.7, 241.4)
- moved R115 3.57 mm to (291.4, 241.4)
- moved R116 3.57 mm to (293.4, 241.4)
- moved R117 3.57 mm to (295.4, 241.4)
- moved R119 3.57 mm to (300.7, 241.4)
- moved C23 3.13 mm to (371.5, 188.3)
- moved C25 3.01 mm to (372.0, 194.7)
- moved C26 2.62 mm to (363.9, 196.8)
- moved C24 2.54 mm to (371.5, 208.6)
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Connections:
- C11 pad 1: +3.3VAnalog -> GNDA
- C11 pad 2: GNDA -> +3.3VAnalog
- C12 pad 1: +3.3VAnalog -> GNDA
- C12 pad 2: GNDA -> +3.3VAnalog
- C25 pad 1: GND -> GNDPWR
- C26 pad 2: GND -> GNDPWR
- C4 pad 1: +3.3VDigital -> GND
- C4 pad 2: GND -> +3.3VDigital
- J3 pad 11: AVRCP_NEXT -> AVRC_PREV
- J3 pad 3: I2C_SDA -> unconnected-(J3-Pin_3-Pad3)
- J3 pad 4: I2C_SCL -> unconnected-(J3-Pin_4-Pad4)
- J3 pad 5: unconnected-(J3-Pin_5-Pad5) -> I2C_SDA
- J3 pad 6: unconnected-(J3-Pin_6-Pad6) -> I2C_SCL
- J3 pad 7: AVRC_PREV -> AVRCP_NEXT
- U2 pad 30: AVRCP_PLAY -> AVRCP_NEXT
- U2 pad 31: AVRCP_NEXT -> AVRCP_PLAY
Routing:
- net Net-(U2-IO35): track 0.00 -> 115.1 mm, vias 0 -> 2
- net Net-(U2-IO34): track 0.00 -> 100.9 mm, vias 0 -> 2
- net Net-(U4B--): track 0.00 -> 99.5 mm, vias 0 -> 4
- net RAHighL: track 0.00 -> 85.3 mm, vias 0 -> 2
- net Net-(U4A--): track 0.00 -> 85.3 mm, vias 0 -> 2
- net LeftFront+: track 0.00 -> 84.1 mm
- net RANCHighL: track 0.00 -> 78.8 mm, vias 0 -> 2
- net RANCHighR: track 0.00 -> 75.7 mm
- net RAMidL: track 0.00 -> 70.1 mm, vias 0 -> 2
- net RAHighR: track 0.00 -> 69.0 mm
- net AVRCP_NEXT: track 0.00 -> 67.7 mm
- net RANCMidL: track 0.00 -> 67.0 mm
- net RANCLowR: track 0.00 -> 66.4 mm, vias 0 -> 2
- net RALowR: track 0.00 -> 64.6 mm, vias 0 -> 2
- net AVRCP_PLAY: track 0.00 -> 63.9 mm
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- added copper zone on F.Cu, net GND
- added copper zone on F.Cu, net GNDA
Other:
- board text added: "Arduino Picko"
- board text added: "Manufactured in Македониjа"
- board text removed: "+"

Commit message: progress sync
Parts:
- moved R127 80.4 mm to (275.6, 284.4)
- moved C107 79.9 mm to (286.0, 275.0)
- moved C108 79.9 mm to (282.3, 282.7)
- moved R123 79.9 mm to (289.3, 278.5)
- moved R124 79.9 mm to (278.9, 277.2)
- moved U27 79.9 mm to (284.2, 278.8)
- moved R126 79.6 mm to (293.4, 281.4)
- moved C103 79.6 mm to (272.4, 282.2)
- moved C104 79.6 mm to (266.9, 290.2)
- moved C105 79.6 mm to (298.4, 282.2)
- moved C106 79.6 mm to (293.4, 290.2)
- moved RV7 79.6 mm to (268.4, 294.8)
- moved RV8 79.6 mm to (294.9, 294.8)
- moved U25 79.6 mm to (269.6, 286.2)
- moved U26 79.6 mm to (295.9, 286.2)
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Connections:
- U8 pad 4: unconnected-(U8-NC-Pad4) -> GND
Routing:
- net MSL: track 3.10 -> 139.6 mm
- net MSR: track 2.95 -> 112.6 mm
- net LeftFront-: track 0.00 -> 97.7 mm, vias 0 -> 2
- net FAL: track 3.16 -> 96.0 mm, vias 0 -> 6
- net FAR: track 2.83 -> 91.4 mm, vias 0 -> 2
- net RightFront-: track 0.00 -> 86.6 mm
- net RightFront+: track 0.00 -> 82.9 mm
- net FANCR: track 0.00 -> 80.9 mm, vias 0 -> 2
- net FANCL: track 0.00 -> 70.1 mm, vias 0 -> 2
- net +5VAnalog: track 0.00 -> 46.1 mm
- net -5VAnalog: track 0.00 -> 45.9 mm
- net Net-(U27B--): track 2.67 -> 33.6 mm, vias 0 -> 4
- net Net-(U27A--): track 2.80 -> 30.9 mm, vias 0 -> 2
- net Net-(C48-Pad1): track 0.00 -> 21.6 mm, vias 0 -> 2
- net +3.3VDigital: track 27.0 -> 46.6 mm
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- added copper zone on F.Cu, net Net-(C48-Pad1)
- added copper zone on F.Cu, net Net-(U6-SW)

Commit message: pcbs done
Parts:
- removed the G*** at (214.1, 159.1)
- added G***: LOGO, LOGO, F.Cu at (276.1, 253.0)
- added G***: LOGO, LOGO, F.Cu at (273.2, 237.6)
- added R134: 10k, Resistor_SMD:R_0805_2012Metric_Pad1.20x1.40mm_HandSolder, F.Cu at (166.4, 295.2)
- added R135: 10k, Resistor_SMD:R_0805_2012Metric_Pad1.20x1.40mm_HandSolder, F.Cu at (177.2, 297.2)
- added REF**: NetTie-2_SMD_Pad2.0mm, NetTie:NetTie-2_SMD_Pad2.0mm, F.Cu at (292.0, 202.8)
- added REF**: MountingHole_2.1mm, MountingHole:MountingHole_2.1mm, F.Cu at (389.5, 147.9)
- added REF**: MountingHole_2.1mm, MountingHole:MountingHole_2.1mm, F.Cu at (389.5, 308.0)
- added REF**: MountingHole_2.1mm, MountingHole:MountingHole_2.1mm, F.Cu at (283.9, 308.0)
- added REF**: MountingHole_2.1mm, MountingHole:MountingHole_2.1mm, F.Cu at (163.0, 147.9)
- added REF**: NetTie-2_SMD_Pad2.0mm, NetTie:NetTie-2_SMD_Pad2.0mm, F.Cu at (294.8, 202.8)
- added REF**: MountingHole_2.1mm, MountingHole:MountingHole_2.1mm, F.Cu at (389.5, 225.8)
- added REF**: MountingHole_2.1mm, MountingHole:MountingHole_2.1mm, F.Cu at (180.1, 308.0)
- R1, R3: value 10k -> 100k
- R7: value 2.7k -> 2k
- moved G*** 46.3 mm to (174.8, 212.4)
- moved U2 28.9 mm to (195.7, 170.4)
- moved J3 28.1 mm to (238.0, 193.1)
- moved IC1 3.09 mm to (392.2, 198.3)
- moved U10 1.48 mm to (332.9, 219.6)
- moved U5 1.38 mm to (307.3, 214.0)
- moved C19 1.38 mm to (304.1, 213.9)
- moved C18 1.38 mm to (310.5, 213.9)
- moved C38 0.51 mm to (309.8, 203.2)
- moved C21 0.50 mm to (313.3, 225.6)
- moved C20 0.40 mm to (313.6, 216.7)
- moved C39 0.40 mm to (309.5, 209.2)
- moved C40 0.40 mm to (313.6, 210.3)
- moved L2 0.40 mm to (317.0, 204.8)
- moved R129 0.40 mm to (313.6, 214.5)
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Connections:
- J6 pad a1: +5VAnalog -> -5VAnalog
- J6 pad a2: -5VAnalog -> +5VAnalog
- U5 pad 4: unconnected-(U5-NC-Pad4) -> GNDA
Routing:
- net +5VAnalog: track 46.1 -> 758.3 mm, vias 0 -> 31
- net -5VAnalog: track 45.9 -> 721.3 mm, vias 0 -> 41
- net +12VPerm: track 3.90 -> 207.3 mm, vias 0 -> 3
- net +3.3VDigital: track 46.6 -> 165.8 mm, vias 0 -> 8
- net RANCL: track 0.00 -> 112.8 mm, vias 0 -> 8
- net RANCR: track 0.00 -> 110.3 mm, vias 0 -> 8
- net +3.3VAnalog: track 11.1 -> 121.2 mm, vias 0 -> 3
- net +5VDigital: track 7.68 -> 116.0 mm, vias 0 -> 2
- net Net-(U2-IO34): track 100.9 -> 132.3 mm, vias 2 -> 4
- net Net-(U2-IO35): track 112.0 -> 143.1 mm
- net GNDA: track 66.9 -> 93.8 mm, vias 0 -> 309
- net Net-(U10-*SHDN): track 0.00 -> 26.0 mm
- net I2S_SCK: track 54.7 -> 80.6 mm
- net I2S_SD: track 22.8 -> 47.5 mm
- net I2S_WS: track 24.9 -> 48.2 mm
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- added copper zone on B.Cu, net +12VPerm
- added copper zone on F.Cu, net +3.3VAnalog
- added copper zone on F.Cu, net +3.3VDigital
- added copper zone on F.Cu, net +5VAnalog
- added copper zone on F.Cu, net -5VAnalog
- added copper zone on B.Cu, net GND
- added copper zone on B.Cu, net GNDA
- added copper zone on B.Cu, net GNDPWR
- added copper zone on F.Cu, net GNDPWR
- added copper zone on F.Cu, net Net-(C40-Pad1)
- added copper zone on F.Cu, net Net-(U7-GND)
- added copper zone on F.Cu, net Net-(U7-SW)
- added copper zone on F.Cu, net Net-(U9-SW)
Other:
- board size 232.1 x 165.8 mm -> 232.1 x 165.7 mm
- board text added: "4 Ohm Speakers"
- board text added: "Arduino Pičko"
- board text added: "Произведено во Света Троица"
- board text removed: "Arduino Picko"
- board text removed: "Manufactured in Македониjа"
