File: Electronics/AudioSystemFull/AudioSystemFull.kicad_pcb (KiCad board)
At the start: 2 copper layers, 232.1 x 165.7 mm, 305 parts, among them IC1 TDA1558Q, J1 SJ1-3515-SMT-TR-BE, J3 Conn_Display_Buttons, J6 Conn_ISO, U1 MIC39100-5.0WS, U10 LT3015EQ-5PBF, U11 OPA2134, U12 OPA2134, U13 OPA2134, U14 OPA2134, U15 OPA2134, U16 OPA2134, U17 OPA2134, U18 OPA2134, U19 OPA2134, U2 DEVKIT_V1_ESP32-WROOM-32, U20 OPA2134, U21 OPA2134, U22 OPA2134, U23 OPA2134, U24 OPA2134, U25 OPA2134, U26 OPA2134, U27 OPA2134, U28 OPA2134, U3 PCM5102A, U4 OPA2134, U5 LP5907MFX-3.3, U6 LMR51420YFDDCR, U7 LMR51420YFDDCR, U8 LP5907MFX-3.3, U9 LMR51420YFDDCR

Commit message: bom
Parts:
- C1, C2, C23, C24: footprint Capacitor_SMD:C_0805_2012Metric_Pad1.18x1.45mm_HandSolder -> Capacitor_SMD:C_1206_3216Metric_Pad1.33x1.80mm_HandSolder
- L1, L3, L6: footprint AudioSystemFootprintLibrary:SRP0315-1R0K -> AudioSystemFootprintLibrary:SRP5030T-1R0M
- moved C23 1.81 mm to (373.3, 188.2)
- moved L6 1.19 mm to (276.2, 196.0)
- moved J1 1.05 mm to (168.7, 303.6)
- moved L1 0.63 mm to (340.4, 194.9)
- moved C1 0.60 mm to (173.4, 294.6)
- moved C2 0.38 mm to (163.2, 294.4)
- moved L3 0.21 mm to (307.4, 195.3)
Routing:
- net Net-(IC1-INPUT1): track 11.4 -> 9.19 mm
- net MSL: track 139.6 -> 140.9 mm
- net Net-(U2-IO34): track 132.3 -> 133.4 mm
- net Net-(C45-Pad1): track 5.93 -> 6.95 mm
- net Net-(C31-Pad1): track 6.23 -> 6.80 mm
- net Net-(IC1-IN3): track 11.4 -> 10.8 mm
- net MSR: track 112.6 -> 112.1 mm
- net GNDA: vias 309 -> 311
