File: Electronics/AudioSystemNoiseCancellationPanel/AudioSystemNoiseCancellationPanel.kicad_pcb (KiCad board)
At the start: 2 copper layers, 21.6 x 15.9 mm, 13 parts, among them J1 Conn_01x04_Pin, U1 OPA134, U2 MIC5365-1.2YC5-TR

Commit message: bom
Parts:
- C2, C4: value 0.1u -> 100n
