File: Electronics/AudioSystemNoiseCancellationPanel/AudioSystemNoiseCancellationPanel.kicad_sch (KiCad schematic)
At the start: 12 parts, among them J1 Conn_01x04_Pin, U1 OPA134, U2 MIC5365-1.2YC5-TR

Commit message: bom
Parts:
- C1, C3: Check_prices (none) -> https://www.mouser.bg/ProductDetail/80-C0805C105K3R?R=80-C0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; MANUFACTURER (none) -> C0805C105K3RACTU; Price (none) -> 0.186
- C2, C4: value 0.1u -> 100n; Check_prices (none) -> https://www.mouser.bg/ProductDetail/KEMET/C0805C104K3RACTU?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; MANUFACTURER (none) -> C0805C104K3RACTU; Price (none) -> 0.186
- C5, C6: Check_prices (none) -> https://www.mouser.bg/ProductDetail/KEMET/C0805C104K3RACTU?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; MANUFACTURER (none) -> C0805C104K3RACTU; Price (none) -> 0.186
- J1: MANUFACTURER (none) -> None; Price (none) -> None
- MK1: Check_prices https://www.snapeda.com/parts/ICS-40310/TDK+InvenSense/view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 -> https://www.mouser.bg/ProductDetail/TDK-InvenSense/ICS-4031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; MANUFACTURER InvenSense -> ICS-40310
- R1: Check_prices (none) -> https://www.mouser.bg/ProductDetail/YAGEO/RT0805DRE0747KL?q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; MANUFACTURER (none) -> RT0805DRE0747KL; Price (none) -> 0.186
- R2: Check_prices (none) -> https://www.mouser.bg/ProductDetail/YAGEO/RT0805FRE07820KL?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; MANUFACTURER (none) -> RT0805FRE07820KL; Price (none) -> 0.186
- U1: Check_prices (none) -> https://www.mouser.bg/ProductDetail/Texas-Instruments/OPA13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; MANUFACTURER (none) -> OPA134UA; Price (none) -> None
- U2: Check_prices https://www.snapeda.com/parts/MIC5365-1.2YC5-TR/Microchip/v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 -> https://www.mouser.bg/ProductDetail/Microchip-Technology/MI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; MANUFACTURER Micrel -> MIC5365-1.2YC5-TR; Price None -> 0.335
